File: peci.kicad_sch (KiCad schematic)
At the start: 0 parts

Commit message: [#99625] Implement PECI schematic
Parts:
- added C401, C405: C_100n_0402, antmicro-footprints:C_0402_1005Metric, symbol antmicroCapacitors0402:C_100n_0402
- added Q401: PJE138K, antmicro-footprints:SOT-523, symbol antmicroTransistorsFETsMOSFETsSingle:PJE138K
- added R401, R403, R404: R_0R_0402, antmicro-footprints:R_0402_1005Metric, symbol antmicroResistors0402:R_0R_0402
- added R402, R405: R_10k_0402, antmicro-footprints:R_0402_1005Metric, symbol antmicroResistors0402:R_10k_0402
- added TP401: TP_0.75mm_SMD, antmicro-footprints:TP_SMD_0.75mm, symbol antmicroTestPoints:TP_0.75mm_SMD
- added U402: MAX6621AUBT, antmicro-footprints:VSSOP-10_3x3mm_P0.5mm, symbol antmicroInterfaceControllers:MAX6621AUBT
Connections:
- new net: Q401.3 (D), R402.1, U402.8 (~{RESET})
- new net: TP401.1, U402.9 (~{ALERT})
- new net: R401.2, U402.3 (AD0)
- new net +1V8: Q401.1 (G), R405.2
- new net +3V3: C405.2, R402.2, U402.6 (VCC)
- new net DC_SCM_PECI: U402.1 (PECI)
- new net GND: C401.1, C405.1, R401.1, U402.2 (AGND), U402.7 (GND)
- new net I2C_3V3.SCL: R404.2
- new net I2C_3V3.SDA: R403.2
- new net PECI_VREF: C401.2, U402.10 (VREF)
- new net SCL: R404.1, U402.5 (SCL)
- new net SDA: R403.1, U402.4 (SDA)
- new net ~{RESET}: Q401.2 (S), R405.1
