File: front-panel-eth.kicad_sch (KiCad schematic)
At the start: 0 parts

Commit message: [#99642] Add KSZ9131RNX PHY. Add ETH RJ45 front panel connector
Parts:
- added C1001: C_100n_0402, antmicro-footprints:C_0402_1005Metric, symbol antmicroCapacitors0402:C_100n_0402
- added J1001: Bus_RJ45_7498111120R, antmicro-footprints:Bus_RJ45_7498111120R, symbol antmicroModularConnectorsJacksWithMagnetics:Bus_RJ45_7498111120R
- added R1001: R_330R_0402, antmicro-footprints:R_0402_1005Metric, symbol antmicroResistors0402:R_330R_0402
- added R1002, R1003: R_470R_0402, antmicro-footprints:R_0402_1005Metric, symbol antmicroResistors0402:R_470R_0402
- added R1004, R1005: R_0R_0402, antmicro-footprints:R_0402_1005Metric, symbol antmicroResistors0402:R_0R_0402
Connections:
- new net: J1001.2 (LED2_G+), R1003.1
- new net: C1001.1, J1001.SH, R1001.1
- new net: J1001.13 (LED1_Y-), R1004.1
- new net: J1001.14 (LED1_Y+), R1002.1
- new net: J1001.1 (LED2_G-), R1005.1
- new net +3V3: R1002.2, R1003.2
- new net ETHERNET.MDI0+: J1001.3 (D1+)
- new net ETHERNET.MDI0-: J1001.4 (D1-)
- new net ETHERNET.MDI1+: J1001.5 (D2+)
- new net ETHERNET.MDI1-: J1001.6 (D2-)
- new net ETHERNET.MDI2+: J1001.7 (D3+)
- new net ETHERNET.MDI2-: J1001.8 (D3-)
- new net ETHERNET.MDI3+: J1001.9 (D4+)
- new net ETHERNET.MDI3-: J1001.10 (D4-)
- new net ETH_LED_G: R1005.2
- new net ETH_LED_Y: R1004.2
- new net GND: C1001.2, J1001.12 (GND), R1001.2
- no-connect marks 0 -> 1
