File: front-panel-eth.kicad_sch (KiCad schematic)
At the start: 7 parts, among them J1001 Bus_RJ45_7498111120R

Commit message: [#100282] Reorder schematic pages, reannotate schematic
Parts:
- renumbered C1001 to C2401, J1001 to J2401, R1002 to R2401, R1003 to R2402, R1004 to R2403, R1005 to R2404, R1001 to R2405
Changed lines of the file:
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@@
 		(in_pos_files yes)
 		(dnp no)
-		(property "Reference" "#PWR01001"
+		(property "Reference" "#PWR02403"
 			(at 182.88 180.34 0)
 			(hide yes)
@@
 			(project "altera-modular-agilex-5-dc-scm"
 				(path "/6bb9d978-a328-4b30-874b-55170a976185/2f6f709e-e133-4af2-b82d-2efdce120bcc"
-					(reference "#PWR01001")
+					(reference "#PWR02403")
 					(unit 1)
 				)
@@
 		(in_pos_files yes)
 		(dnp no)
-		(property "Reference" "#PWR01003"
+		(property "Reference" "#PWR02405"
 			(at 208.28 184.15 0)
 			(hide yes)
@@
 			(project "altera-modular-agilex-5-dc-scm"
 				(path "/6bb9d978-a328-4b30-874b-55170a976185/2f6f709e-e133-4af2-b82d-2efdce120bcc"
-					(reference "#PWR01003")
+					(reference "#PWR02405")
 					(unit 1)
 				)
@@
 		(dnp no)
 		(fields_autoplaced yes)
-		(property "Reference" "R1003"
+		(property "Reference" "R2402"
 			(at 260.35 133.35 90)
 			(show_name no)
@@
 			(project "altera-modular-agilex-5-dc-scm"
 				(path "/6bb9d978-a328-4b30-874b-55170a976185/2f6f709e-e133-4af2-b82d-2efdce120bcc"
-					(reference "R1003")
+					(reference "R2402")
 					(unit 1)
 				)
@@
 		(dnp no)
 		(fields_autoplaced yes)
-		(property "Reference" "R1001"
+		(property "Reference" "R2405"
 			(at 210.82 172.72 90)
 			(show_name no)
@@
 			(project "altera-modular-agilex-5-dc-scm"
 				(path "/6bb9d978-a328-4b30-874b-55170a976185/2f6f709e-e133-4af2-b82d-2efdce120bcc"
-					(reference "R1001")
+					(reference "R2405")
 					(unit 1)
 				)
@@
 		(in_pos_files yes)
 		(dnp no)
-		(property "Reference" "R1004"
+		(property "Reference" "R2403"
 			(at 262.89 139.954 0)
 			(show_name no)
@@
 			(project "altera-modular-agilex-5-dc-scm"
 				(path "/6bb9d978-a328-4b30-874b-55170a976185/2f6f709e-e133-4af2-b82d-2efdce120bcc"
-					(reference "R1004")
+					(reference "R2403")
 					(unit 1)
 				)
@@
 		(dnp no)
 		(fields_autoplaced yes)
-		(property "Reference" "C1001"
+		(property "Reference" "C2401"
 			(at 199.39 172.7263 90)
 			(show_name no)
@@
 			(project "altera-modular-agilex-5-dc-scm"
 				(path "/6bb9d978-a328-4b30-874b-55170a976185/2f6f709e-e133-4af2-b82d-2efdce120bcc"
-					(reference "C1001")
+					(reference "C2401")
 					(unit 1)
 				)
@@
 		(dnp no)
 		(fields_autoplaced yes)
-		(property "Reference" "R1002"
+		(property "Reference" "R2401"
 			(at 248.92 133.35 90)
 			(show_name no)
@@
 			(project "altera-modular-agilex-5-dc-scm"
 				(path "/6bb9d978-a328-4b30-874b-55170a976185/2f6f709e-e133-4af2-b82d-2efdce120bcc"
-					(reference "R1002")
+					(reference "R2401")
 					(unit 1)
 				)
@@
 		(in_pos_files yes)
 		(dnp no)
-		(property "Reference" "#PWR01004"
+		(property "Reference" "#PWR02401"
 			(at 261.62 129.54 0)
 			(hide yes)
@@
 			(project "altera-modular-agilex-5-dc-scm"
 				(path "/6bb9d978-a328-4b30-874b-55170a976185/2f6f709e-e133-4af2-b82d-2efdce120bcc"
-					(reference "#PWR01004")
+					(reference "#PWR02401")
 					(unit 1)
 				)
@@
 		(in_pos_files yes)
 		(dnp no)
-		(property "Reference" "#PWR01005"
+		(property "Reference" "#PWR02402"
 			(at 273.05 129.54 0)
 			(hide yes)
@@
 			(project "altera-modular-agilex-5-dc-scm"
 				(path "/6bb9d978-a328-4b30-874b-55170a976185/2f6f709e-e133-4af2-b82d-2efdce120bcc"
-					(reference "#PWR01005")
+					(reference "#PWR02402")
 					(unit 1)
 				)
@@
 		(in_pos_files yes)
 		(dnp no)
-		(property "Reference" "R1005"
+		(property "Reference" "R2404"
 			(at 262.89 147.574 0)
 			(show_name no)
@@
 			(project "altera-modular-agilex-5-dc-scm"
 				(path "/6bb9d978-a328-4b30-874b-55170a976185/2f6f709e-e133-4af2-b82d-2efdce120bcc"
-					(reference "R1005")
+					(reference "R2404")
 					(unit 1)
 				)
@@
 		(dnp no)
 		(fields_autoplaced yes)
-		(property "Reference" "J1001"
+		(property "Reference" "J2401"
 			(at 229.87 132.08 0)
 			(show_name no)
@@
 			(project "altera-modular-agilex-5-dc-scm"
 				(path "/6bb9d978-a328-4b30-874b-55170a976185/2f6f709e-e133-4af2-b82d-2efdce120bcc"
-					(reference "J1001")
+					(reference "J2401")
 					(unit 1)
 				)
@@
 		(in_pos_files yes)
 		(dnp no)
-		(property "Reference" "#PWR01002"
+		(property "Reference" "#PWR02404"
 			(at 196.85 184.15 0)
 			(hide yes)
@@
 			(project "altera-modular-agilex-5-dc-scm"
 				(path "/6bb9d978-a328-4b30-874b-55170a976185/2f6f709e-e133-4af2-b82d-2efdce120bcc"
-					(reference "#PWR01002")
+					(reference "#PWR02404")
 					(unit 1)
 				)
