File: front-panel-eth.kicad_sch (KiCad schematic)
At the start: 7 parts, among them J2401 Bus_RJ45_7498111120R

Commit message: [#100282] Add missing schematic sheet names and align them all
Changed lines of the file:
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@@
 	(text "Front panel ETH"
 		(exclude_from_sim no)
-		(at 203.2 38.1 0)
+		(at 210.82 38.1 0)
 		(effects
 			(font

Commit message: [#100501] Reannotate schematic
Parts:
- renumbered C2401 to C243, J2401 to J11, R2401 to R306, R2402 to R307, R2403 to R308, R2404 to R309, R2405 to R310
Changed lines of the file:
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@@
 		(in_pos_files yes)
 		(dnp no)
-		(property "Reference" "#PWR02403"
+		(property "Reference" "#PWR0425"
 			(at 168.91 184.15 0)
 			(hide yes)
@@
 			(project "altera-modular-agilex-5-dc-scm"
 				(path "/6bb9d978-a328-4b30-874b-55170a976185/2f6f709e-e133-4af2-b82d-2efdce120bcc"
-					(reference "#PWR02403")
+					(reference "#PWR0425")
 					(unit 1)
 				)
@@
 		(in_pos_files yes)
 		(dnp no)
-		(property "Reference" "#PWR02405"
+		(property "Reference" "#PWR0427"
 			(at 194.31 187.96 0)
 			(hide yes)
@@
 			(project "altera-modular-agilex-5-dc-scm"
 				(path "/6bb9d978-a328-4b30-874b-55170a976185/2f6f709e-e133-4af2-b82d-2efdce120bcc"
-					(reference "#PWR02405")
+					(reference "#PWR0427")
 					(unit 1)
 				)
@@
 		(dnp no)
 		(fields_autoplaced yes)
-		(property "Reference" "R2402"
+		(property "Reference" "R307"
 			(at 246.38 137.16 90)
 			(show_name no)
@@
 			(project "altera-modular-agilex-5-dc-scm"
 				(path "/6bb9d978-a328-4b30-874b-55170a976185/2f6f709e-e133-4af2-b82d-2efdce120bcc"
-					(reference "R2402")
+					(reference "R307")
 					(unit 1)
 				)
@@
 		(dnp no)
 		(fields_autoplaced yes)
-		(property "Reference" "R2405"
+		(property "Reference" "R310"
 			(at 196.85 176.53 90)
 			(show_name no)
@@
 			(project "altera-modular-agilex-5-dc-scm"
 				(path "/6bb9d978-a328-4b30-874b-55170a976185/2f6f709e-e133-4af2-b82d-2efdce120bcc"
-					(reference "R2405")
+					(reference "R310")
 					(unit 1)
 				)
@@
 		(in_pos_files yes)
 		(dnp no)
-		(property "Reference" "R2403"
+		(property "Reference" "R308"
 			(at 248.92 143.764 0)
 			(show_name no)
@@
 			(project "altera-modular-agilex-5-dc-scm"
 				(path "/6bb9d978-a328-4b30-874b-55170a976185/2f6f709e-e133-4af2-b82d-2efdce120bcc"
-					(reference "R2403")
+					(reference "R308")
 					(unit 1)
 				)
@@
 		(dnp no)
 		(fields_autoplaced yes)
-		(property "Reference" "C2401"
+		(property "Reference" "C243"
 			(at 185.42 176.5363 90)
 			(show_name no)
@@
 			(project "altera-modular-agilex-5-dc-scm"
 				(path "/6bb9d978-a328-4b30-874b-55170a976185/2f6f709e-e133-4af2-b82d-2efdce120bcc"
-					(reference "C2401")
+					(reference "C243")
 					(unit 1)
 				)
@@
 		(dnp no)
 		(fields_autoplaced yes)
-		(property "Reference" "R2401"
+		(property "Reference" "R306"
 			(at 234.95 137.16 90)
 			(show_name no)
@@
 			(project "altera-modular-agilex-5-dc-scm"
 				(path "/6bb9d978-a328-4b30-874b-55170a976185/2f6f709e-e133-4af2-b82d-2efdce120bcc"
-					(reference "R2401")
+					(reference "R306")
 					(unit 1)
 				)
@@
 		(in_pos_files yes)
 		(dnp no)
-		(property "Reference" "#PWR02401"
+		(property "Reference" "#PWR0423"
 			(at 247.65 133.35 0)
 			(hide yes)
@@
 			(project "altera-modular-agilex-5-dc-scm"
 				(path "/6bb9d978-a328-4b30-874b-55170a976185/2f6f709e-e133-4af2-b82d-2efdce120bcc"
-					(reference "#PWR02401")
+					(reference "#PWR0423")
 					(unit 1)
 				)
@@
 		(in_pos_files yes)
 		(dnp no)
-		(property "Reference" "#PWR02402"
+		(property "Reference" "#PWR0424"
 			(at 259.08 133.35 0)
 			(hide yes)
@@
 			(project "altera-modular-agilex-5-dc-scm"
 				(path "/6bb9d978-a328-4b30-874b-55170a976185/2f6f709e-e133-4af2-b82d-2efdce120bcc"
-					(reference "#PWR02402")
+					(reference "#PWR0424")
 					(unit 1)
 				)
@@
 		(in_pos_files yes)
 		(dnp no)
-		(property "Reference" "R2404"
+		(property "Reference" "R309"
 			(at 248.92 151.384 0)
 			(show_name no)
@@
 			(project "altera-modular-agilex-5-dc-scm"
 				(path "/6bb9d978-a328-4b30-874b-55170a976185/2f6f709e-e133-4af2-b82d-2efdce120bcc"
-					(reference "R2404")
+					(reference "R309")
 					(unit 1)
 				)
@@
 		(dnp no)
 		(fields_autoplaced yes)
-		(property "Reference" "J2401"
+		(property "Reference" "J11"
 			(at 215.9 135.89 0)
 			(show_name no)
@@
 			(project "altera-modular-agilex-5-dc-scm"
 				(path "/6bb9d978-a328-4b30-874b-55170a976185/2f6f709e-e133-4af2-b82d-2efdce120bcc"
-					(reference "J2401")
+					(reference "J11")
 					(unit 1)
 				)
@@
 		(in_pos_files yes)
 		(dnp no)
-		(property "Reference" "#PWR02404"
+		(property "Reference" "#PWR0426"
 			(at 182.88 187.96 0)
 			(hide yes)
@@
 			(project "altera-modular-agilex-5-dc-scm"
 				(path "/6bb9d978-a328-4b30-874b-55170a976185/2f6f709e-e133-4af2-b82d-2efdce120bcc"
-					(reference "#PWR02404")
+					(reference "#PWR0426")
 					(unit 1)
 				)

Commit message: [#100501] Reannotate schematic
Parts:
- renumbered C243 to C235, J11 to J13, R306 to R338, R307 to R339, R308 to R340, R309 to R341, R310 to R342
Changed lines of the file:
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@@
 		(in_pos_files yes)
 		(dnp no)
-		(property "Reference" "#PWR0425"
+		(property "Reference" "#PWR0417"
 			(at 168.91 184.15 0)
 			(hide yes)
@@
 			(project "altera-modular-agilex-5-dc-scm"
 				(path "/6bb9d978-a328-4b30-874b-55170a976185/2f6f709e-e133-4af2-b82d-2efdce120bcc"
-					(reference "#PWR0425")
+					(reference "#PWR0417")
 					(unit 1)
 				)
@@
 		(in_pos_files yes)
 		(dnp no)
-		(property "Reference" "#PWR0427"
+		(property "Reference" "#PWR0419"
 			(at 194.31 187.96 0)
 			(hide yes)
@@
 			(project "altera-modular-agilex-5-dc-scm"
 				(path "/6bb9d978-a328-4b30-874b-55170a976185/2f6f709e-e133-4af2-b82d-2efdce120bcc"
-					(reference "#PWR0427")
+					(reference "#PWR0419")
 					(unit 1)
 				)
@@
 		(dnp no)
 		(fields_autoplaced yes)
-		(property "Reference" "R307"
+		(property "Reference" "R339"
 			(at 246.38 137.16 90)
 			(show_name no)
@@
 			(project "altera-modular-agilex-5-dc-scm"
 				(path "/6bb9d978-a328-4b30-874b-55170a976185/2f6f709e-e133-4af2-b82d-2efdce120bcc"
-					(reference "R307")
+					(reference "R339")
 					(unit 1)
 				)
@@
 		(dnp no)
 		(fields_autoplaced yes)
-		(property "Reference" "R310"
+		(property "Reference" "R342"
 			(at 196.85 176.53 90)
 			(show_name no)
@@
 			(project "altera-modular-agilex-5-dc-scm"
 				(path "/6bb9d978-a328-4b30-874b-55170a976185/2f6f709e-e133-4af2-b82d-2efdce120bcc"
-					(reference "R310")
+					(reference "R342")
 					(unit 1)
 				)
@@
 		(in_pos_files yes)
 		(dnp no)
-		(property "Reference" "R308"
+		(property "Reference" "R340"
 			(at 248.92 143.764 0)
 			(show_name no)
@@
 			(project "altera-modular-agilex-5-dc-scm"
 				(path "/6bb9d978-a328-4b30-874b-55170a976185/2f6f709e-e133-4af2-b82d-2efdce120bcc"
-					(reference "R308")
+					(reference "R340")
 					(unit 1)
 				)
@@
 		(dnp no)
 		(fields_autoplaced yes)
-		(property "Reference" "C243"
+		(property "Reference" "C235"
 			(at 185.42 176.5363 90)
 			(show_name no)
@@
 			(project "altera-modular-agilex-5-dc-scm"
 				(path "/6bb9d978-a328-4b30-874b-55170a976185/2f6f709e-e133-4af2-b82d-2efdce120bcc"
-					(reference "C243")
+					(reference "C235")
 					(unit 1)
 				)
@@
 		(dnp no)
 		(fields_autoplaced yes)
-		(property "Reference" "R306"
+		(property "Reference" "R338"
 			(at 234.95 137.16 90)
 			(show_name no)
@@
 			(project "altera-modular-agilex-5-dc-scm"
 				(path "/6bb9d978-a328-4b30-874b-55170a976185/2f6f709e-e133-4af2-b82d-2efdce120bcc"
-					(reference "R306")
+					(reference "R338")
 					(unit 1)
 				)
@@
 		(in_pos_files yes)
 		(dnp no)
-		(property "Reference" "#PWR0423"
+		(property "Reference" "#PWR0415"
 			(at 247.65 133.35 0)
 			(hide yes)
@@
 			(project "altera-modular-agilex-5-dc-scm"
 				(path "/6bb9d978-a328-4b30-874b-55170a976185/2f6f709e-e133-4af2-b82d-2efdce120bcc"
-					(reference "#PWR0423")
+					(reference "#PWR0415")
 					(unit 1)
 				)
@@
 		(in_pos_files yes)
 		(dnp no)
-		(property "Reference" "#PWR0424"
+		(property "Reference" "#PWR0416"
 			(at 259.08 133.35 0)
 			(hide yes)
@@
 			(project "altera-modular-agilex-5-dc-scm"
 				(path "/6bb9d978-a328-4b30-874b-55170a976185/2f6f709e-e133-4af2-b82d-2efdce120bcc"
-					(reference "#PWR0424")
+					(reference "#PWR0416")
 					(unit 1)
 				)
@@
 		(in_pos_files yes)
 		(dnp no)
-		(property "Reference" "R309"
+		(property "Reference" "R341"
 			(at 248.92 151.384 0)
 			(show_name no)
@@
 			(project "altera-modular-agilex-5-dc-scm"
 				(path "/6bb9d978-a328-4b30-874b-55170a976185/2f6f709e-e133-4af2-b82d-2efdce120bcc"
-					(reference "R309")
+					(reference "R341")
 					(unit 1)
 				)
@@
 		(dnp no)
 		(fields_autoplaced yes)
-		(property "Reference" "J11"
+		(property "Reference" "J13"
 			(at 215.9 135.89 0)
 			(show_name no)
@@
 			(project "altera-modular-agilex-5-dc-scm"
 				(path "/6bb9d978-a328-4b30-874b-55170a976185/2f6f709e-e133-4af2-b82d-2efdce120bcc"
-					(reference "J11")
+					(reference "J13")
 					(unit 1)
 				)
@@
 		(in_pos_files yes)
 		(dnp no)
-		(property "Reference" "#PWR0426"
+		(property "Reference" "#PWR0418"
 			(at 182.88 187.96 0)
 			(hide yes)
@@
 			(project "altera-modular-agilex-5-dc-scm"
 				(path "/6bb9d978-a328-4b30-874b-55170a976185/2f6f709e-e133-4af2-b82d-2efdce120bcc"
-					(reference "#PWR0426")
+					(reference "#PWR0418")
 					(unit 1)
 				)
