File: eth.kicad_sch (KiCad schematic)
At the start: 58 parts, among them U501 KSZ9131RNXC, Y502 Resonator_25MHz_ECX-1247Q

Commit message: [#99781] Update mismatached component values
Parts:
- R511, R512, R513, R514, R515, R516, R517, R518, R519, R520: value R_2k2_0402 -> R_1k_0402
Changed lines of the file:
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@@
 			(justify right bottom)
 		)
-		(property "Net Class" "100Ohm-diff"
+		(property "Netclass" "100Ohm-diff"
 			(at 260.35 130.81 0)
 			(show_name no)
@@
 			)
 		)
-		(property "Value" "R_2k2_0402"
+		(property "Value" "R_1k_0402"
 			(at 241.3 228.6 0)
 			(hide yes)
@@
 			)
 		)
-		(property "Value" "R_2k2_0402"
+		(property "Value" "R_1k_0402"
 			(at 241.3 236.22 0)
 			(hide yes)
@@
 			)
 		)
-		(property "Value" "R_2k2_0402"
+		(property "Value" "R_1k_0402"
 			(at 241.3 242.57 0)
 			(hide yes)
@@
 			)
 		)
-		(property "Value" "R_2k2_0402"
+		(property "Value" "R_1k_0402"
 			(at 241.3 240.03 0)
 			(hide yes)
@@
 			)
 		)
-		(property "Value" "R_2k2_0402"
+		(property "Value" "R_1k_0402"
 			(at 241.3 255.27 0)
 			(hide yes)
@@
 			)
 		)
-		(property "Value" "R_2k2_0402"
+		(property "Value" "R_1k_0402"
 			(at 241.3 252.73 0)
 			(hide yes)
@@
 			)
 		)
-		(property "Value" "R_2k2_0402"
+		(property "Value" "R_1k_0402"
 			(at 241.3 248.92 0)
 			(hide yes)
@@
 			)
 		)
-		(property "Value" "R_2k2_0402"
+		(property "Value" "R_1k_0402"
 			(at 241.3 231.14 0)
 			(hide yes)
@@
 			)
 		)
-		(property "Value" "R_2k2_0402"
+		(property "Value" "R_1k_0402"
 			(at 241.3 245.11 0)
 			(hide yes)
@@
 			)
 		)
-		(property "Value" "R_2k2_0402"
+		(property "Value" "R_1k_0402"
 			(at 241.3 233.68 0)
 			(hide yes)
