File: pcie-clk.kicad_sch (KiCad schematic)
At the start: 2 parts, among them U1701 SY75602BTWL-TR

Commit message: [#99871] Add clock generator
Parts:
- added C1702, C1703, C1704, C1705, C1706, C1707, C1714: C_1u_0402, antmicro-footprints:C_0402_1005Metric, symbol antmicroCapacitors0402:C_1u_0402
- added C1708, C1709, C1710, C1711, C1712, C1713: C_100n_0402, antmicro-footprints:C_0402_1005Metric, symbol antmicroCapacitors0402:C_100n_0402
- added R1701: R_10k_0402, antmicro-footprints:R_0402_1005Metric, symbol antmicroResistors0402:R_10k_0402
- added R1702, R1703, R1704, R1705: R_0R_0402, antmicro-footprints:R_0402_1005Metric, symbol antmicroResistors0402:R_0R_0402
- added TP1701, TP1702, TP1703: TP_0.75mm_SMD, antmicro-footprints:TP_SMD_0.75mm, symbol antmicroTestPoints:TP_0.75mm_SMD
- added U1702: SI5338B-B-GM, antmicro-footprints:QFN-24-1EP_4x4mm_P0.5_EP2.5x2.5mm, symbol antmicroClockTimingClockGeneratorsPLLsFrequencySynthesizers:SI5338B-B-GM
- added U1703: LMK1C1102DQFT, antmicro-footprints:WSON-8_2x2mm, symbol antmicroClockTimingClockGeneratorsPLLsFrequencySynthesizers:LMK1C1102DQFT
Connections:
- net GND: now also C1702.1, C1703.1, C1704.1, C1705.1, C1706.1, C1707.1, C1714.1, U1702.2 (IN2/CLKINB), U1702.23 (RSVD_GND), U1702.25 (GND), U1702.4 (IN4/I2C_LSB), U1702.6 (IN6/FDBKB), U1703.4 (GND)
- net SOM_CLK.CLK+: now also R1702.2, R1705.1; no longer U1701.6 (OUT1_P)
- net SOM_CLK.CLK-: now also R1703.2, R1704.1; no longer U1701.7 (OUT1_N)
- new net +1V8: C1702.2, C1703.2, C1704.2, C1705.2, C1706.2, C1707.2, C1714.2, R1701.2, U1702.11 (VDDO3), U1702.15 (VDDO2), U1702.16 (VDDO1), U1702.20 (VDDO0), U1702.24 (VDD), U1702.7 (VDD), U1703.6 (VDD)
- new net 100MHz_CLK+: C1712.1, U1702.14 (CLK2A)
- new net 100MHz_CLK-: C1713.1, U1702.13 (CLK2B)
- new net 100MHz_CLK.+: C1712.2, R1705.2
- new net 100MHz_CLK.-: C1713.2, R1704.2
- new net 150MHz_CLK+: C1708.1, U1702.22 (CLK0A)
- new net 150MHz_CLK-: C1709.1, U1702.21 (CLK0B)
- new net 150MHz_CLK.+: C1708.2
- new net 150MHz_CLK.-: C1709.2
- new net 156_25MHz_CLK+: C1710.1, U1702.18 (CLK1A)
- new net 156_25MHz_CLK-: C1711.1, U1702.17 (CLK1B)
- new net 156_25MHz_CLK.+: C1710.2
- new net 156_25MHz_CLK.-: C1711.2
- new net 20MHz_CLK.+: U1702.10 (CLK3A)
- new net 20MHz_CLK.-: U1702.9 (CLK3B)
- new net CLK_25MHz: TP1701.1, U1703.1 (CLKIN)
- new net HPS_CLK_25MHz: TP1702.1, U1703.3 (Y0)
- new net I3C.SCL: U1702.12 (SCL)
- new net I3C.SDA: U1702.19 (SDA)
- new net OUT_EN: R1701.1, U1703.2 (1G)
- new net PLL_CLK_25MHz: TP1703.1, U1702.3 (IN3/CLKIN), U1703.8 (Y1)
- new net SOM_CLK+: R1702.1, U1701.6 (OUT1_P)
- new net SOM_CLK-: R1703.1, U1701.7 (OUT1_N)
- no-connect marks 0 -> 3
Other:
- note added: "Clock generator"
- moved on the sheet: C1701, U1701
