File: ltpi_bias.kicad_sch (KiCad schematic)
At the start: 18 parts

Commit message: [#100282] Reorder schematic pages, reannotate schematic
Parts:
- renumbered C1801 to C1301, C1810 to C1302, C1802 to C1303, C1803 to C1304, C1804 to C1305, C1805 to C1306, C1806 to C1307, C1808 to C1308, C1807 to C1309, C1809 to C1310, R1801 to R1301, R1807 to R1302, R1802 to R1303, R1808 to R1304, R1803 to R1305, R1804 to R1306, R1805 to R1307, R1806 to R1308
Changed lines of the file:
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@@
 			(justify left bottom)
 		)
-		(property "Netclass" "100Ohm-diff"
+		(property "Net Class" "100Ohm-diff"
 			(at 149.098 132.08 0)
 			(show_name no)
@@
 			(justify right bottom)
 		)
-		(property "Netclass" "100Ohm-diff"
+		(property "Net Class" "100Ohm-diff"
 			(at 273.812 132.08 0)
 			(show_name no)
@@
 		(in_pos_files yes)
 		(dnp no)
-		(property "Reference" "#PWR01801"
+		(property "Reference" "#PWR01301"
 			(at 200.66 101.6 0)
 			(hide yes)
@@
 			(project "altera-modular-agilex-5-dc-scm"
 				(path "/6bb9d978-a328-4b30-874b-55170a976185/65eda2d2-086a-48f2-af4e-47077a805913"
-					(reference "#PWR01801")
+					(reference "#PWR01301")
 					(unit 1)
 				)
@@
 		(dnp no)
 		(fields_autoplaced yes)
-		(property "Reference" "C1803"
+		(property "Reference" "C1304"
 			(at 207.0163 133.35 0)
 			(show_name no)
@@
 			(project "altera-modular-agilex-5-dc-scm"
 				(path "/6bb9d978-a328-4b30-874b-55170a976185/65eda2d2-086a-48f2-af4e-47077a805913"
-					(reference "C1803")
+					(reference "C1304")
 					(unit 1)
 				)
@@
 		(dnp no)
 		(fields_autoplaced yes)
-		(property "Reference" "C1802"
+		(property "Reference" "C1303"
 			(at 207.0163 118.11 0)
 			(show_name no)
@@
 			(project "altera-modular-agilex-5-dc-scm"
 				(path "/6bb9d978-a328-4b30-874b-55170a976185/65eda2d2-086a-48f2-af4e-47077a805913"
-					(reference "C1802")
+					(reference "C1303")
 					(unit 1)
 				)
@@
 		(dnp no)
 		(fields_autoplaced yes)
-		(property "Reference" "C1805"
+		(property "Reference" "C1306"
 			(at 207.0163 160.02 0)
 			(show_name no)
@@
 			(project "altera-modular-agilex-5-dc-scm"
 				(path "/6bb9d978-a328-4b30-874b-55170a976185/65eda2d2-086a-48f2-af4e-47077a805913"
-					(reference "C1805")
+					(reference "C1306")
 					(unit 1)
 				)
@@
 		(dnp no)
 		(fields_autoplaced yes)
-		(property "Reference" "C1804"
+		(property "Reference" "C1305"
 			(at 207.0163 144.78 0)
 			(show_name no)
@@
 			(project "altera-modular-agilex-5-dc-scm"
 				(path "/6bb9d978-a328-4b30-874b-55170a976185/65eda2d2-086a-48f2-af4e-47077a805913"
-					(reference "C1804")
+					(reference "C1305")
 					(unit 1)
 				)
@@
 		(in_pos_files yes)
 		(dnp no)
-		(property "Reference" "R1804"
+		(property "Reference" "R1306"
 			(at 218.44 134.62 90)
 			(show_name no)
@@
 			(project "altera-modular-agilex-5-dc-scm"
 				(path "/6bb9d978-a328-4b30-874b-55170a976185/65eda2d2-086a-48f2-af4e-47077a805913"
-					(reference "R1804")
+					(reference "R1306")
 					(unit 1)
 				)
@@
 		(in_pos_files yes)
 		(dnp no)
-		(property "Reference" "#PWR01804"
+		(property "Reference" "#PWR01304"
 			(at 234.95 116.84 0)
 			(hide yes)
@@
 			(project "altera-modular-agilex-5-dc-scm"
 				(path "/6bb9d978-a328-4b30-874b-55170a976185/65eda2d2-086a-48f2-af4e-47077a805913"
-					(reference "#PWR01804")
+					(reference "#PWR01304")
 					(unit 1)
 				)
@@
 		(dnp no)
 		(fields_autoplaced yes)
-		(property "Reference" "C1807"
+		(property "Reference" "C1309"
 			(at 207.0163 182.88 0)
 			(show_name no)
@@
 			(project "altera-modular-agilex-5-dc-scm"
 				(path "/6bb9d978-a328-4b30-874b-55170a976185/65eda2d2-086a-48f2-af4e-47077a805913"
-					(reference "C1807")
+					(reference "C1309")
 					(unit 1)
 				)
@@
 		(in_pos_files yes)
 		(dnp no)
-		(property "Reference" "R1805"
+		(property "Reference" "R1307"
 			(at 218.44 153.67 90)
 			(show_name no)
@@
 			(project "altera-modular-agilex-5-dc-scm"
 				(path "/6bb9d978-a328-4b30-874b-55170a976185/65eda2d2-086a-48f2-af4e-47077a805913"
-					(reference "R1805")
+					(reference "R1307")
 					(unit 1)
 				)
@@
 		(in_pos_files yes)
 		(dnp no)
-		(property "Reference" "R1806"
+		(property "Reference" "R1308"
 			(at 218.44 161.29 90)
 			(show_name no)
@@
 			(project "altera-modular-agilex-5-dc-scm"
 				(path "/6bb9d978-a328-4b30-874b-55170a976185/65eda2d2-086a-48f2-af4e-47077a805913"
-					(reference "R1806")
+					(reference "R1308")
 					(unit 1)
 				)
@@
 		(dnp no)
 		(fields_autoplaced yes)
-		(property "Reference" "C1806"
+		(property "Reference" "C1307"
 			(at 207.0163 172.72 0)
 			(show_name no)
@@
 			(project "altera-modular-agilex-5-dc-scm"
 				(path "/6bb9d978-a328-4b30-874b-55170a976185/65eda2d2-086a-48f2-af4e-47077a805913"
-					(reference "C1806")
+					(reference "C1307")
 					(unit 1)
 				)
@@
 		(dnp no)
 		(fields_autoplaced yes)
-		(property "Reference" "R1802"
+		(property "Reference" "R1303"
 			(at 187.96 107.95 90)
 			(show_name no)
@@
 			(project "altera-modular-agilex-5-dc-scm"
 				(path "/6bb9d978-a328-4b30-874b-55170a976185/65eda2d2-086a-48f2-af4e-47077a805913"
-					(reference "R1802")
+					(reference "R1303")
 					(unit 1)
 				)
@@
 		(in_pos_files yes)
 		(dnp no)
-		(property "Reference" "#PWR01803"
+		(property "Reference" "#PWR01302"
 			(at 241.3 101.6 0)
 			(hide yes)
@@
 			(project "altera-modular-agilex-5-dc-scm"
 				(path "/6bb9d978-a328-4b30-874b-55170a976185/65eda2d2-086a-48f2-af4e-47077a805913"
-					(reference "#PWR01803")
+					(reference "#PWR01302")
 					(unit 1)
 				)
@@
 		(in_pos_files yes)
 		(dnp no)
-		(property "Reference" "R1803"
+		(property "Reference" "R1305"
 			(at 218.44 127 90)
 			(show_name no)
@@
 			(project "altera-modular-agilex-5-dc-scm"
 				(path "/6bb9d978-a328-4b30-874b-55170a976185/65eda2d2-086a-48f2-af4e-47077a805913"
-					(reference "R1803")
+					(reference "R1305")
 					(unit 1)
 				)
@@
 		(dnp no)
 		(fields_autoplaced yes)
-		(property "Reference" "R1801"
+		(property "Reference" "R1301"
 			(at 187.96 100.33 90)
 			(show_name no)
@@
 			(project "altera-modular-agilex-5-dc-scm"
 				(path "/6bb9d978-a328-4b30-874b-55170a976185/65eda2d2-086a-48f2-af4e-47077a805913"
-					(reference "R1801")
+					(reference "R1301")
 					(unit 1)
 				)
@@
 		(dnp no)
 		(fields_autoplaced yes)
-		(property "Reference" "C1809"
+		(property "Reference" "C1310"
 			(at 214.6363 187.96 0)
 			(show_name no)
@@
 			(project "altera-modular-agilex-5-dc-scm"
 				(path "/6bb9d978-a328-4b30-874b-55170a976185/65eda2d2-086a-48f2-af4e-47077a805913"
-					(reference "C1809")
+					(reference "C1310")
 					(unit 1)
 				)
@@
 		(dnp no)
 		(fields_autoplaced yes)
-		(property "Reference" "C1808"
+		(property "Reference" "C1308"
 			(at 214.6363 177.8 0)
 			(show_name no)
@@
 			(project "altera-modular-agilex-5-dc-scm"
 				(path "/6bb9d978-a328-4b30-874b-55170a976185/65eda2d2-086a-48f2-af4e-47077a805913"
-					(reference "C1808")
+					(reference "C1308")
 					(unit 1)
 				)
@@
 		(dnp no)
 		(fields_autoplaced yes)
-		(property "Reference" "R1807"
+		(property "Reference" "R1302"
 			(at 228.6 100.33 90)
 			(show_name no)
@@
 			(project "altera-modular-agilex-5-dc-scm"
 				(path "/6bb9d978-a328-4b30-874b-55170a976185/65eda2d2-086a-48f2-af4e-47077a805913"
-					(reference "R1807")
+					(reference "R1302")
 					(unit 1)
 				)
@@
 		(dnp no)
 		(fields_autoplaced yes)
-		(property "Reference" "C1801"
+		(property "Reference" "C1301"
 			(at 198.12 107.9436 90)
 			(show_name no)
@@
 			(project "altera-modular-agilex-5-dc-scm"
 				(path "/6bb9d978-a328-4b30-874b-55170a976185/65eda2d2-086a-48f2-af4e-47077a805913"
-					(reference "C1801")
+					(reference "C1301")
 					(unit 1)
 				)
@@
 		(dnp no)
 		(fields_autoplaced yes)
-		(property "Reference" "C1810"
+		(property "Reference" "C1302"
 			(at 238.76 107.9436 90)
 			(show_name no)
@@
 			(project "altera-modular-agilex-5-dc-scm"
 				(path "/6bb9d978-a328-4b30-874b-55170a976185/65eda2d2-086a-48f2-af4e-47077a805913"
-					(reference "C1810")
+					(reference "C1302")
 					(unit 1)
 				)
@@
 		(in_pos_files yes)
 		(dnp no)
-		(property "Reference" "#PWR01802"
+		(property "Reference" "#PWR01303"
 			(at 194.31 116.84 0)
 			(hide yes)
@@
 			(project "altera-modular-agilex-5-dc-scm"
 				(path "/6bb9d978-a328-4b30-874b-55170a976185/65eda2d2-086a-48f2-af4e-47077a805913"
-					(reference "#PWR01802")
+					(reference "#PWR01303")
 					(unit 1)
 				)
@@
 		(dnp no)
 		(fields_autoplaced yes)
-		(property "Reference" "R1808"
+		(property "Reference" "R1304"
 			(at 228.6 107.95 90)
 			(show_name no)
@@
 			(project "altera-modular-agilex-5-dc-scm"
 				(path "/6bb9d978-a328-4b30-874b-55170a976185/65eda2d2-086a-48f2-af4e-47077a805913"
-					(reference "R1808")
+					(reference "R1304")
 					(unit 1)
 				)
