File: ltpi_bias.kicad_sch (KiCad schematic)
At the start: 18 parts

Commit message: [#100501] Perform minor BOM consolidation
Parts:
- C95, C96: value C_100n_16V_X7R_0402 -> C_100n_0402; symbol antmicroCapacitors0402:C_100n_16V_X7R_0402 -> antmicroCapacitors0402:C_100n_0402; Dielectric X7R -> X5R; MPN C0402C104J4RAC7411 -> GRM155R61H104KE14D; Manufacturer KEMET -> Murata; Voltage 16V -> 50V
Changed lines of the file:
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@@
 	)
 	(symbol
-		(lib_id "antmicroCapacitors0402:C_100n_16V_X7R_0402")
+		(lib_id "antmicroCapacitors0402:C_100n_0402")
 		(at 195.58 111.76 90)
 		(unit 1)
@@
 			)
 		)
-		(property "Value" "C_100n_16V_X7R_0402"
+		(property "Value" "C_100n_0402"
 			(at 218.44 96.52 0)
 			(hide yes)
@@
 			)
 		)
-		(property "Datasheet" "https://www.kemet.com/en/us/capacitors/product/C0402C104J4RAC7411.html"
+		(property "Datasheet" "https://www.murata.com/products/productdetail?partno=GRM155R61H104KE14%23"
 			(at 223.52 96.52 0)
 			(hide yes)
@@
 			)
 		)
-		(property "Description" "SMD Multilayer Ceramic Capacitor, 100nF, 16V, 0402, ±5%, X7R"
+		(property "Description" "SMD Multilayer Ceramic Capacitor, 0.1 µF, 50 V, 0402 [1005 Metric], ± 10%, X5R, GRM Series"
 			(at 195.58 111.76 0)
 			(hide yes)
@@
 			)
 		)
-		(property "MPN" "C0402C104J4RAC7411"
+		(property "MPN" "GRM155R61H104KE14D"
 			(at 226.06 96.52 0)
 			(hide yes)
@@
 			)
 		)
-		(property "Voltage" "16V"
+		(property "Voltage" "50V"
 			(at 205.74 96.52 0)
 			(hide yes)
@@
 			)
 		)
-		(property "Dielectric" "X7R"
+		(property "Dielectric" "X5R"
 			(at 208.28 96.52 0)
 			(hide yes)
@@
 			)
 		)
-		(property "Manufacturer" "KEMET"
+		(property "Manufacturer" "Murata"
 			(at 210.82 96.52 0)
 			(hide yes)
@@
 	)
 	(symbol
-		(lib_id "antmicroCapacitors0402:C_100n_16V_X7R_0402")
+		(lib_id "antmicroCapacitors0402:C_100n_0402")
 		(at 236.22 111.76 90)
 		(unit 1)
@@
 			)
 		)
-		(property "Value" "C_100n_16V_X7R_0402"
+		(property "Value" "C_100n_0402"
 			(at 259.08 96.52 0)
 			(hide yes)
@@
 			)
 		)
-		(property "Datasheet" "https://www.kemet.com/en/us/capacitors/product/C0402C104J4RAC7411.html"
+		(property "Datasheet" "https://www.murata.com/products/productdetail?partno=GRM155R61H104KE14%23"
 			(at 264.16 96.52 0)
 			(hide yes)
@@
 			)
 		)
-		(property "Description" "SMD Multilayer Ceramic Capacitor, 100nF, 16V, 0402, ±5%, X7R"
+		(property "Description" "SMD Multilayer Ceramic Capacitor, 0.1 µF, 50 V, 0402 [1005 Metric], ± 10%, X5R, GRM Series"
 			(at 236.22 111.76 0)
 			(hide yes)
@@
 			)
 		)
-		(property "MPN" "C0402C104J4RAC7411"
+		(property "MPN" "GRM155R61H104KE14D"
 			(at 266.7 96.52 0)
 			(hide yes)
@@
 			)
 		)
-		(property "Voltage" "16V"
+		(property "Voltage" "50V"
 			(at 246.38 96.52 0)
 			(hide yes)
@@
 			)
 		)
-		(property "Dielectric" "X7R"
+		(property "Dielectric" "X5R"
 			(at 248.92 96.52 0)
 			(hide yes)
@@
 			)
 		)
-		(property "Manufacturer" "KEMET"
+		(property "Manufacturer" "Murata"
 			(at 251.46 96.52 0)
 			(hide yes)
