File: sd-card.kicad_sch (KiCad schematic)
At the start: 13 parts, among them J901 MicroSD_1140084168, U901 LSF0108RKSR

Commit message: [#100282] Reorder schematic pages, reannotate schematic
Parts:
- renumbered C901 to C1101, C902 to C1102, C903 to C1103, J901 to J1101, R901 to R1101, R902 to R1102, R903 to R1103, R904 to R1104, R905 to R1105, R906 to R1106, R907 to R1107, R908 to R1108, U901 to U1101
Changed lines of the file:
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@@
 		(in_pos_files yes)
 		(dnp no)
-		(property "Reference" "#PWR0909"
+		(property "Reference" "#PWR01105"
 			(at 170.18 175.26 0)
 			(hide yes)
@@
 			(project "altera-modular-agilex-5-dc-scm"
 				(path "/6bb9d978-a328-4b30-874b-55170a976185/e62a0a22-c003-4281-aacf-cd65a22f5da7"
-					(reference "#PWR0909")
+					(reference "#PWR01105")
 					(unit 1)
 				)
@@
 		(in_pos_files yes)
 		(dnp no)
-		(property "Reference" "R907"
+		(property "Reference" "R1107"
 			(at 243.84 133.35 90)
 			(show_name no)
@@
 			(project "altera-modular-agilex-5-dc-scm"
 				(path "/6bb9d978-a328-4b30-874b-55170a976185/e62a0a22-c003-4281-aacf-cd65a22f5da7"
-					(reference "R907")
+					(reference "R1107")
 					(unit 1)
 				)
@@
 		(in_pos_files yes)
 		(dnp no)
-		(property "Reference" "#PWR0908"
+		(property "Reference" "#PWR01107"
 			(at 259.08 175.26 0)
 			(hide yes)
@@
 			(project "altera-modular-agilex-5-dc-scm"
 				(path "/6bb9d978-a328-4b30-874b-55170a976185/e62a0a22-c003-4281-aacf-cd65a22f5da7"
-					(reference "#PWR0908")
+					(reference "#PWR01107")
 					(unit 1)
 				)
@@
 		(in_pos_files yes)
 		(dnp no)
-		(property "Reference" "#PWR0907"
+		(property "Reference" "#PWR01108"
 			(at 265.43 175.26 0)
 			(hide yes)
@@
 			(project "altera-modular-agilex-5-dc-scm"
 				(path "/6bb9d978-a328-4b30-874b-55170a976185/e62a0a22-c003-4281-aacf-cd65a22f5da7"
-					(reference "#PWR0907")
+					(reference "#PWR01108")
 					(unit 1)
 				)
@@
 		(in_pos_files yes)
 		(dnp no)
-		(property "Reference" "R901"
+		(property "Reference" "R1101"
 			(at 193.04 124.714 0)
 			(show_name no)
@@
 			(project "altera-modular-agilex-5-dc-scm"
 				(path "/6bb9d978-a328-4b30-874b-55170a976185/e62a0a22-c003-4281-aacf-cd65a22f5da7"
-					(reference "R901")
+					(reference "R1101")
 					(unit 1)
 				)
@@
 		(in_pos_files yes)
 		(dnp no)
-		(property "Reference" "R902"
+		(property "Reference" "R1102"
 			(at 199.39 133.35 90)
 			(show_name no)
@@
 			(project "altera-modular-agilex-5-dc-scm"
 				(path "/6bb9d978-a328-4b30-874b-55170a976185/e62a0a22-c003-4281-aacf-cd65a22f5da7"
-					(reference "R902")
+					(reference "R1102")
 					(unit 1)
 				)
@@
 		(in_pos_files yes)
 		(dnp no)
-		(property "Reference" "#PWR0904"
+		(property "Reference" "#PWR01101"
 			(at 168.91 127 0)
 			(hide yes)
@@
 			(project "altera-modular-agilex-5-dc-scm"
 				(path "/6bb9d978-a328-4b30-874b-55170a976185/e62a0a22-c003-4281-aacf-cd65a22f5da7"
-					(reference "#PWR0904")
+					(reference "#PWR01101")
 					(unit 1)
 				)
@@
 		(in_pos_files yes)
 		(dnp no)
-		(property "Reference" "C901"
+		(property "Reference" "C1101"
 			(at 153.162 128.778 90)
 			(show_name no)
@@
 			(project "altera-modular-agilex-5-dc-scm"
 				(path "/6bb9d978-a328-4b30-874b-55170a976185/e62a0a22-c003-4281-aacf-cd65a22f5da7"
-					(reference "C901")
+					(reference "C1101")
 					(unit 1)
 				)
@@
 		(in_pos_files yes)
 		(dnp no)
-		(property "Reference" "C902"
+		(property "Reference" "C1102"
 			(at 183.388 128.778 90)
 			(show_name no)
@@
 			(project "altera-modular-agilex-5-dc-scm"
 				(path "/6bb9d978-a328-4b30-874b-55170a976185/e62a0a22-c003-4281-aacf-cd65a22f5da7"
-					(reference "C902")
+					(reference "C1102")
 					(unit 1)
 				)
@@
 		(in_pos_files yes)
 		(dnp no)
-		(property "Reference" "#PWR0903"
+		(property "Reference" "#PWR01106"
 			(at 189.23 175.26 0)
 			(hide yes)
@@
 			(project "altera-modular-agilex-5-dc-scm"
 				(path "/6bb9d978-a328-4b30-874b-55170a976185/e62a0a22-c003-4281-aacf-cd65a22f5da7"
-					(reference "#PWR0903")
+					(reference "#PWR01106")
 					(unit 1)
 				)
@@
 		(in_pos_files yes)
 		(dnp no)
-		(property "Reference" "C903"
+		(property "Reference" "C1103"
 			(at 249.682 166.878 90)
 			(show_name no)
@@
 			(project "altera-modular-agilex-5-dc-scm"
 				(path "/6bb9d978-a328-4b30-874b-55170a976185/e62a0a22-c003-4281-aacf-cd65a22f5da7"
-					(reference "C903")
+					(reference "C1103")
 					(unit 1)
 				)
@@
 		(in_pos_files yes)
 		(dnp no)
-		(property "Reference" "#PWR0901"
+		(property "Reference" "#PWR01109"
 			(at 294.64 175.26 0)
 			(hide yes)
@@
 			(project "altera-modular-agilex-5-dc-scm"
 				(path "/6bb9d978-a328-4b30-874b-55170a976185/e62a0a22-c003-4281-aacf-cd65a22f5da7"
-					(reference "#PWR0901")
+					(reference "#PWR01109")
 					(unit 1)
 				)
@@
 		(dnp no)
 		(fields_autoplaced yes)
-		(property "Reference" "J901"
+		(property "Reference" "J1101"
 			(at 274.955 138.43 0)
 			(show_name no)
@@
 			(project "altera-modular-agilex-5-dc-scm"
 				(path "/6bb9d978-a328-4b30-874b-55170a976185/e62a0a22-c003-4281-aacf-cd65a22f5da7"
-					(reference "J901")
+					(reference "J1101")
 					(unit 1)
 				)
@@
 		(in_pos_files yes)
 		(dnp no)
-		(property "Reference" "R904"
+		(property "Reference" "R1104"
 			(at 217.17 133.35 90)
 			(show_name no)
@@
 			(project "altera-modular-agilex-5-dc-scm"
 				(path "/6bb9d978-a328-4b30-874b-55170a976185/e62a0a22-c003-4281-aacf-cd65a22f5da7"
-					(reference "R904")
+					(reference "R1104")
 					(unit 1)
 				)
@@
 		(in_pos_files yes)
 		(dnp no)
-		(property "Reference" "#PWR0906"
+		(property "Reference" "#PWR01104"
 			(at 191.77 137.16 0)
 			(hide yes)
@@
 			(project "altera-modular-agilex-5-dc-scm"
 				(path "/6bb9d978-a328-4b30-874b-55170a976185/e62a0a22-c003-4281-aacf-cd65a22f5da7"
-					(reference "#PWR0906")
+					(reference "#PWR01104")
 					(unit 1)
 				)
@@
 		(in_pos_files yes)
 		(dnp no)
-		(property "Reference" "R905"
+		(property "Reference" "R1105"
 			(at 226.06 133.35 90)
 			(show_name no)
@@
 			(project "altera-modular-agilex-5-dc-scm"
 				(path "/6bb9d978-a328-4b30-874b-55170a976185/e62a0a22-c003-4281-aacf-cd65a22f5da7"
-					(reference "R905")
+					(reference "R1105")
 					(unit 1)
 				)
@@
 		(in_pos_files yes)
 		(dnp no)
-		(property "Reference" "#PWR0902"
+		(property "Reference" "#PWR01102"
 			(at 265.43 124.46 0)
 			(hide yes)
@@
 			(project "altera-modular-agilex-5-dc-scm"
 				(path "/6bb9d978-a328-4b30-874b-55170a976185/e62a0a22-c003-4281-aacf-cd65a22f5da7"
-					(reference "#PWR0902")
+					(reference "#PWR01102")
 					(unit 1)
 				)
@@
 		(in_pos_files yes)
 		(dnp no)
-		(property "Reference" "#PWR0905"
+		(property "Reference" "#PWR01103"
 			(at 144.78 137.16 0)
 			(hide yes)
@@
 			(project "altera-modular-agilex-5-dc-scm"
 				(path "/6bb9d978-a328-4b30-874b-55170a976185/e62a0a22-c003-4281-aacf-cd65a22f5da7"
-					(reference "#PWR0905")
+					(reference "#PWR01103")
 					(unit 1)
 				)
@@
 		(dnp no)
 		(fields_autoplaced yes)
-		(property "Reference" "U901"
+		(property "Reference" "U1101"
 			(at 168.275 132.08 0)
 			(show_name no)
@@
 			(project "altera-modular-agilex-5-dc-scm"
 				(path "/6bb9d978-a328-4b30-874b-55170a976185/e62a0a22-c003-4281-aacf-cd65a22f5da7"
-					(reference "U901")
+					(reference "U1101")
 					(unit 1)
 				)
@@
 		(in_pos_files yes)
 		(dnp no)
-		(property "Reference" "R906"
+		(property "Reference" "R1106"
 			(at 234.95 133.35 90)
 			(show_name no)
@@
 			(project "altera-modular-agilex-5-dc-scm"
 				(path "/6bb9d978-a328-4b30-874b-55170a976185/e62a0a22-c003-4281-aacf-cd65a22f5da7"
-					(reference "R906")
+					(reference "R1106")
 					(unit 1)
 				)
@@
 		(in_pos_files yes)
 		(dnp no)
-		(property "Reference" "R903"
+		(property "Reference" "R1103"
 			(at 208.28 133.35 90)
 			(show_name no)
@@
 			(project "altera-modular-agilex-5-dc-scm"
 				(path "/6bb9d978-a328-4b30-874b-55170a976185/e62a0a22-c003-4281-aacf-cd65a22f5da7"
-					(reference "R903")
+					(reference "R1103")
 					(unit 1)
 				)
@@
 		(in_pos_files yes)
 		(dnp no)
-		(property "Reference" "R908"
+		(property "Reference" "R1108"
 			(at 156.21 175.26 90)
 			(show_name no)
@@
 			(project "altera-modular-agilex-5-dc-scm"
 				(path "/6bb9d978-a328-4b30-874b-55170a976185/e62a0a22-c003-4281-aacf-cd65a22f5da7"
-					(reference "R908")
+					(reference "R1108")
 					(unit 1)
 				)
