File: ulpi-phy.kicad_sch (KiCad schematic)
At the start: 16 parts, among them U1501 USB3320C-EZK-TR, Y1503 Resonator_24MHz_ECX-1247

Commit message: [#100282] Reorder schematic pages, reannotate schematic
Parts:
- renumbered C1508 to C1701, C1504 to C1702, C1503 to C1703, C1502 to C1704, C1501 to C1705, C1506 to C1706, C1505 to C1707, C1507 to C1708, R1501 to R1701, R1507 to R1702, R1503 to R1703, R1504 to R1704, R1502 to R1705, TP1501 to TP1701, U1501 to U1701, Y1503 to Y1701
