File: ulpi-phy.kicad_sch (KiCad schematic)
At the start: 16 parts, among them U1701 USB3320C-EZK-TR, Y1701 Resonator_24MHz_ECX-1247

Commit message: [#100282] Fix overlaping graphics, add schematic sheet names on them
Other:
- note added: "ULPI PHY"
Changed lines of the file:
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@@
 		(company "Altera")
+	)
+	(text "ULPI PHY"
+		(exclude_from_sim no)
+		(at 203.2 38.1 0)
+		(effects
+			(font
+				(size 4 4)
+				(thickness 0.8)
+				(bold yes)
+			)
+		)
 	)
 	(junction
