File: usb-hub.kicad_sch (KiCad schematic)
At the start: 23 parts, among them U701 USB2422-I_MJ, Y701 Resonator_24MHz_ECX-1247

Commit message: [#100282] Reorder schematic pages, reannotate schematic
Parts:
- renumbered C707 to C1601, C706 to C1602, C705 to C1603, C704 to C1604, C702 to C1605, C701 to C1606, C703 to C1607, C708 to C1608, C709 to C1609, R704 to R1601, R701 to R1602, R705 to R1603, R706 to R1604, R708 to R1605, R716 to R1606, R707 to R1607, R717 to R1608, R715 to R1609, R713 to R1610, R709 to R1611, R714 to R1612, U701 to U1601, Y701 to Y1601
