File: usb-hub.kicad_sch (KiCad schematic)
At the start: 23 parts, among them U1601 USB2422-I_MJ, Y1601 Resonator_24MHz_ECX-1247

Commit message: [#100501] Reannotate schematic
Parts:
- renumbered C1601 to C130, C1602 to C131, C1603 to C132, C1604 to C133, C1605 to C134, C1606 to C135, C1607 to C136, C1608 to C137, C1609 to C138, R1601 to R166, R1602 to R167, R1603 to R168, R1604 to R169, R1605 to R170, R1606 to R171, R1607 to R172, R1608 to R173, R1609 to R174, R1610 to R175, R1611 to R176, R1612 to R177, U1601 to U21, Y1601 to Y2

Commit message: [#100501] Fix USB Hub strap option for non-removable ports
Connections:
- net NON_REM0: now also R175.1; no longer R177.2
- net NON_REM1: now also R177.2; no longer R175.1
Changed lines of the file:
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@@
+		)
+	)
+	(label "NON_REM0"
+		(at 203.2 205.74 0)
+		(effects
+			(font
+				(size 1.27 1.27)
+			)
+			(justify left bottom)
 		)
 	)
@@
 		)
 	)
-	(label "NON_REM0"
+	(label "NON_REM1"
 		(at 203.2 210.82 0)
 		(effects
@@
 		(effects
 			(font
-				(size 1.27 1.27)
-			)
-			(justify left bottom)
-		)
-	)
-	(label "NON_REM1"
-		(at 203.2 205.74 0)
-		(effects
-			(font

Commit message: [#100501] Connect ULPI CPEN signal to USB hub VBUS_DET
Parts:
- removed C133: C_1u_0402, antmicro-footprints:C_0402_1005Metric, symbol antmicroCapacitors0402:C_1u_0402
- removed R166: R_10k_0402, antmicro-footprints:R_0402_1005Metric, symbol antmicroResistors0402:R_10k_0402

Commit message: [#100501] Reannotate schematic
Parts:
- renumbered C130 to C136, C131 to C137, C132 to C138, C134 to C139, C135 to C140, C136 to C141, C137 to C142, C138 to C143, R167 to R212, R168 to R213, R169 to R214, R170 to R215, R171 to R216, R172 to R217, R173 to R218, R174 to R219, R175 to R220, R176 to R221, R177 to R222, U21 to U20

Commit message: [#100501] Perform minor BOM consolidation
Parts:
- C136, C137, C138, C139, C143: value C_1u_0402 -> C_1u_25V_0402; symbol antmicroCapacitors0402:C_1u_0402 -> antmicroCapacitors0402:C_1u_25V_0402; Dielectric (none) -> X5R; MPN C1005X6S1A105K050BC -> GRM155R61E105KE11J; Manufacturer TDK -> Murata; Voltage (none) -> 25V
Changed lines of the file:
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@@
 	)
 	(symbol
-		(lib_id "antmicroCapacitors0402:C_1u_0402")
+		(lib_id "antmicroCapacitors0402:C_1u_25V_0402")
 		(at 185.42 118.11 270)
 		(mirror x)
@@
 			)
 		)
-		(property "Value" "C_1u_0402"
+		(property "Value" "C_1u_25V_0402"
 			(at 175.26 97.79 0)
 			(hide yes)
@@
 			)
 		)
-		(property "Datasheet" "https://product.tdk.com/en/search/capacitor/ceramic/mlcc/info?part_no=C1005X6S1A105K050BC"
+		(property "Datasheet" "https://www.murata.com/products/productdetail?partno=GRM155R61E105KE11%23"
 			(at 170.18 97.79 0)
 			(hide yes)
@@
 			)
 		)
-		(property "Description" "SMD Multilayer Ceramic Capacitor, 1 µF, 10 V, 0402 [1005 Metric], ± 10%, X6S, C"
+		(property "Description" "SMD Multilayer Ceramic Capacitor, 1 µF, 25 V, 0402 [1005 Metric], ± 10%, X5R, GRM Series"
 			(at 152.4 97.79 0)
 			(hide yes)
@@
 			)
 		)
-		(property "MPN" "C1005X6S1A105K050BC"
+		(property "MPN" "GRM155R61E105KE11J"
 			(at 167.64 97.79 0)
 			(hide yes)
@@
 			)
 		)
-		(property "Manufacturer" "TDK"
+		(property "Manufacturer" "Murata"
 			(at 165.1 97.79 0)
 			(hide yes)
@@
 			)
 		)
-		(property "Voltage" ""
+		(property "Voltage" "25V"
 			(at 157.48 97.79 0)
 			(hide yes)
@@
 			)
 		)
-		(property "Dielectric" ""
+		(property "Dielectric" "X5R"
 			(at 154.94 97.79 0)
 			(hide yes)
@@
 	)
 	(symbol
-		(lib_id "antmicroCapacitors0402:C_1u_0402")
+		(lib_id "antmicroCapacitors0402:C_1u_25V_0402")
 		(at 167.64 118.11 270)
 		(mirror x)
@@
 			)
 		)
-		(property "Value" "C_1u_0402"
+		(property "Value" "C_1u_25V_0402"
 			(at 157.48 97.79 0)
 			(hide yes)
@@
 			)
 		)
-		(property "Datasheet" "https://product.tdk.com/en/search/capacitor/ceramic/mlcc/info?part_no=C1005X6S1A105K050BC"
+		(property "Datasheet" "https://www.murata.com/products/productdetail?partno=GRM155R61E105KE11%23"
 			(at 152.4 97.79 0)
 			(hide yes)
@@
 			)
 		)
-		(property "Description" "SMD Multilayer Ceramic Capacitor, 1 µF, 10 V, 0402 [1005 Metric], ± 10%, X6S, C"
+		(property "Description" "SMD Multilayer Ceramic Capacitor, 1 µF, 25 V, 0402 [1005 Metric], ± 10%, X5R, GRM Series"
 			(at 134.62 97.79 0)
 			(hide yes)
@@
 			)
 		)
-		(property "MPN" "C1005X6S1A105K050BC"
+		(property "MPN" "GRM155R61E105KE11J"
 			(at 149.86 97.79 0)
 			(hide yes)
@@
 			)
 		)
-		(property "Manufacturer" "TDK"
+		(property "Manufacturer" "Murata"
 			(at 147.32 97.79 0)
 			(hide yes)
@@
 			)
 		)
-		(property "Voltage" ""
+		(property "Voltage" "25V"
 			(at 139.7 97.79 0)
 			(hide yes)
@@
 			)
 		)
-		(property "Dielectric" ""
+		(property "Dielectric" "X5R"
 			(at 137.16 97.79 0)
 			(hide yes)
@@
 	)
 	(symbol
-		(lib_id "antmicroCapacitors0402:C_1u_0402")
+		(lib_id "antmicroCapacitors0402:C_1u_25V_0402")
 		(at 176.53 118.11 270)
 		(mirror x)
@@
 			)
 		)
-		(property "Value" "C_1u_0402"
+		(property "Value" "C_1u_25V_0402"
 			(at 166.37 97.79 0)
 			(hide yes)
@@
 			)
 		)
-		(property "Datasheet" "https://product.tdk.com/en/search/capacitor/ceramic/mlcc/info?part_no=C1005X6S1A105K050BC"
+		(property "Datasheet" "https://www.murata.com/products/productdetail?partno=GRM155R61E105KE11%23"
 			(at 161.29 97.79 0)
 			(hide yes)
@@
 			)
 		)
-		(property "Description" "SMD Multilayer Ceramic Capacitor, 1 µF, 10 V, 0402 [1005 Metric], ± 10%, X6S, C"
+		(property "Description" "SMD Multilayer Ceramic Capacitor, 1 µF, 25 V, 0402 [1005 Metric], ± 10%, X5R, GRM Series"
 			(at 143.51 97.79 0)
 			(hide yes)
@@
 			)
 		)
-		(property "MPN" "C1005X6S1A105K050BC"
+		(property "MPN" "GRM155R61E105KE11J"
 			(at 158.75 97.79 0)
 			(hide yes)
@@
 			)
 		)
-		(property "Manufacturer" "TDK"
+		(property "Manufacturer" "Murata"
 			(at 156.21 97.79 0)
 			(hide yes)
@@
 			)
 		)
-		(property "Voltage" ""
+		(property "Voltage" "25V"
 			(at 148.59 97.79 0)
 			(hide yes)
@@
 			)
 		)
-		(property "Dielectric" ""
+		(property "Dielectric" "X5R"
 			(at 146.05 97.79 0)
 			(hide yes)
@@
 	)
 	(symbol
-		(lib_id "antmicroCapacitors0402:C_1u_0402")
+		(lib_id "antmicroCapacitors0402:C_1u_25V_0402")
 		(at 156.21 120.65 270)
 		(mirror x)
@@
 			)
 		)
-		(property "Value" "C_1u_0402"
+		(property "Value" "C_1u_25V_0402"
 			(at 146.05 100.33 0)
 			(hide yes)
@@
 			)
 		)
-		(property "Datasheet" "https://product.tdk.com/en/search/capacitor/ceramic/mlcc/info?part_no=C1005X6S1A105K050BC"
+		(property "Datasheet" "https://www.murata.com/products/productdetail?partno=GRM155R61E105KE11%23"
 			(at 140.97 100.33 0)
 			(hide yes)
@@
 			)
 		)
-		(property "Description" "SMD Multilayer Ceramic Capacitor, 1 µF, 10 V, 0402 [1005 Metric], ± 10%, X6S, C"
+		(property "Description" "SMD Multilayer Ceramic Capacitor, 1 µF, 25 V, 0402 [1005 Metric], ± 10%, X5R, GRM Series"
 			(at 156.21 120.65 0)
 			(hide yes)
@@
 			)
 		)
-		(property "MPN" "C1005X6S1A105K050BC"
+		(property "MPN" "GRM155R61E105KE11J"
 			(at 138.43 100.33 0)
 			(hide yes)
@@
 			)
 		)
-		(property "Manufacturer" "TDK"
+		(property "Manufacturer" "Murata"
 			(at 135.89 100.33 0)
 			(hide yes)
@@
 			)
 		)
-		(property "Voltage" ""
+		(property "Voltage" "25V"
 			(at 128.27 100.33 0)
 			(hide yes)
@@
 			)
 		)
-		(property "Dielectric" ""
+		(property "Dielectric" "X5R"
 			(at 125.73 100.33 0)
 			(hide yes)
@@
 	)
 	(symbol
-		(lib_id "antmicroCapacitors0402:C_1u_0402")
+		(lib_id "antmicroCapacitors0402:C_1u_25V_0402")
 		(at 247.65 168.91 90)
 		(unit 1)
@@
 			)
 		)
-		(property "Value" "C_1u_0402"
+		(property "Value" "C_1u_25V_0402"
 			(at 257.81 148.59 0)
 			(hide yes)
@@
 			)
 		)
-		(property "Datasheet" "https://product.tdk.com/en/search/capacitor/ceramic/mlcc/info?part_no=C1005X6S1A105K050BC"
+		(property "Datasheet" "https://www.murata.com/products/productdetail?partno=GRM155R61E105KE11%23"
 			(at 262.89 148.59 0)
 			(hide yes)
@@
 			)
 		)
-		(property "Description" "SMD Multilayer Ceramic Capacitor, 1 µF, 10 V, 0402 [1005 Metric], ± 10%, X6S, C"
+		(property "Description" "SMD Multilayer Ceramic Capacitor, 1 µF, 25 V, 0402 [1005 Metric], ± 10%, X5R, GRM Series"
 			(at 280.67 148.59 0)
 			(hide yes)
@@
 			)
 		)
-		(property "MPN" "C1005X6S1A105K050BC"
+		(property "MPN" "GRM155R61E105KE11J"
 			(at 265.43 148.59 0)
 			(hide yes)
@@
 			)
 		)
-		(property "Manufacturer" "TDK"
+		(property "Manufacturer" "Murata"
 			(at 267.97 148.59 0)
 			(hide yes)
@@
 			)
 		)
-		(property "Voltage" ""
+		(property "Voltage" "25V"
 			(at 275.59 148.59 0)
 			(hide yes)
@@
 			)
 		)
-		(property "Dielectric" ""
+		(property "Dielectric" "X5R"
 			(at 278.13 148.59 0)
 			(hide yes)
