File: mitysom-config.kicad_sch (KiCad schematic)
At the start: 1 part, among them J2701 Plug_Samtec_SEAM-50-02.0-L-08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

Commit message: [#100282] Reorder schematic pages, reannotate schematic
Parts:
- renumbered J2701 to J201
Changed lines of the file:
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@@
 		(dnp no)
 		(fields_autoplaced yes)
-		(property "Reference" "J2701"
+		(property "Reference" "J201"
 			(at 222.25 147.3199 0)
 			(show_name no)
@@
 			(project "altera-modular-agilex-5-dc-scm"
 				(path "/6bb9d978-a328-4b30-874b-55170a976185/44f62d5f-99b7-4265-9c30-e48dbfd6f996"
-					(reference "J2701")
+					(reference "J201")
 					(unit 8)
 				)

Commit message: [#100282] Change SoM connector designator to J100
Parts:
- renumbered J201 to J100
Other:
- note removed: "CONFIG"
Changed lines of the file:
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@@
-		)
-	)
-	(text "CONFIG"
-		(exclude_from_sim no)
-		(at 210.566 168.91 0)
-		(effects
-			(font
-				(size 1.27 1.27)
-			)
 		)
 	)
@@
 		(dnp no)
 		(fields_autoplaced yes)
-		(property "Reference" "J201"
+		(property "Reference" "J100"
 			(at 222.25 147.3199 0)
 			(show_name no)
@@
 			(project "altera-modular-agilex-5-dc-scm"
 				(path "/6bb9d978-a328-4b30-874b-55170a976185/44f62d5f-99b7-4265-9c30-e48dbfd6f996"
-					(reference "J201")
+					(reference "J100")
 					(unit 8)
 				)
