File: mitysom-config.kicad_sch (KiCad schematic)
At the start: 1 part, among them J100 Plug_Samtec_SEAM-50-02.0-L-08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

Commit message: [#100282] Add missing schematic sheet names and align them all
Changed lines of the file:
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@@
 	(text "MitySOM-A5E Mini\nConfig"
 		(exclude_from_sim no)
-		(at 203.2 38.1 0)
+		(at 210.82 38.1 0)
 		(effects
 			(font

Commit message: [#100501] Gate GbE_PHY_RESET with COLD_RESET signal, to reset ETH PHY
Connections:
- net ~{RESET_BTN} renamed ~{HPS_COLD_RESET}
Changed lines of the file:
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@@
 		)
 	)
-	(hierarchical_label "~{RESET_BTN}"
+	(hierarchical_label "~{HPS_COLD_RESET}"
 		(shape input)
 		(at 195.58 157.48 180)
