File: mitysom-hsio.kicad_sch (KiCad schematic)
At the start: 2 parts, among them J2401 Plug_Samtec_SEAM-50-02.0-L-08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

Commit message: [#100282] Reorder schematic pages, reannotate schematic
Parts:
- renumbered J2401 to J401, R2401 to R401
Changed lines of the file:
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@@
 		(in_pos_files yes)
 		(dnp no)
-		(property "Reference" "R2401"
+		(property "Reference" "R401"
 			(at 182.88 151.13 0)
 			(show_name no)
@@
 			(project "altera-modular-agilex-5-dc-scm"
 				(path "/6bb9d978-a328-4b30-874b-55170a976185/266bf6db-77fc-4e99-b82f-dd347350f420"
-					(reference "R2401")
+					(reference "R401")
 					(unit 1)
 				)
@@
 		(dnp no)
 		(fields_autoplaced yes)
-		(property "Reference" "J2401"
+		(property "Reference" "J401"
 			(at 210.185 120.65 0)
 			(show_name no)
@@
 			(project "altera-modular-agilex-5-dc-scm"
 				(path "/6bb9d978-a328-4b30-874b-55170a976185/266bf6db-77fc-4e99-b82f-dd347350f420"
-					(reference "J2401")
+					(reference "J401")
 					(unit 4)
 				)
@@
 		(in_pos_files yes)
 		(dnp no)
-		(property "Reference" "#PWR02401"
+		(property "Reference" "#PWR0401"
 			(at 172.72 153.67 0)
 			(hide yes)
@@
 			(project "altera-modular-agilex-5-dc-scm"
 				(path "/6bb9d978-a328-4b30-874b-55170a976185/266bf6db-77fc-4e99-b82f-dd347350f420"
-					(reference "#PWR02401")
+					(reference "#PWR0401")
 					(unit 1)
 				)

Commit message: [#100282] Change SoM connector designator to J100
Parts:
- renumbered J401 to J100
Changed lines of the file:
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@@
 		(dnp no)
 		(fields_autoplaced yes)
-		(property "Reference" "J401"
+		(property "Reference" "J100"
 			(at 210.185 120.65 0)
 			(show_name no)
@@
 			(project "altera-modular-agilex-5-dc-scm"
 				(path "/6bb9d978-a328-4b30-874b-55170a976185/266bf6db-77fc-4e99-b82f-dd347350f420"
-					(reference "J401")
+					(reference "J100")
 					(unit 4)
 				)
