File: mitysom-hsio.kicad_sch (KiCad schematic)
At the start: 2 parts, among them J100 Plug_Samtec_SEAM-50-02.0-L-08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

Commit message: [#100282] WIP: Clear ERC
Connections:
- no-connect marks 0 -> 13
Changed lines of the file:
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@@
 		)
+	)
+	(no_connect
+		(at 186.69 149.86)
+	)
+	(no_connect
+		(at 186.69 156.21)
+	)
+	(no_connect
+		(at 186.69 128.27)
+	)
+	(no_connect
+		(at 233.68 137.16)
+	)
+	(no_connect
+		(at 233.68 147.32)
+	)
+	(no_connect
+		(at 233.68 143.51)
+	)
+	(no_connect
+		(at 233.68 134.62)
+	)
+	(no_connect
+		(at 233.68 140.97)
+	)
+	(no_connect
+		(at 233.68 149.86)
+	)
+	(no_connect
+		(at 186.69 140.97)
+	)
+	(no_connect
+		(at 186.69 147.32)
+	)
+	(no_connect
+		(at 186.69 143.51)
+	)
+	(no_connect
+		(at 186.69 130.81)
 	)
 	(bus_entry
