File: mitysom-hsio.kicad_sch (KiCad schematic)
At the start: 2 parts, among them J100 Plug_Samtec_SEAM-50-02.0-L-08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

Commit message: [#100282] Add missing schematic sheet names and align them all
Changed lines of the file:
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@@
 	(text "MitySOM-A5E Mini\nHSIO"
 		(exclude_from_sim no)
-		(at 203.2 38.1 0)
+		(at 210.82 38.1 0)
 		(effects
 			(font

Commit message: [#100501] Reannotate schematic
Parts:
- renumbered J100 to J1, R401 to R9
Changed lines of the file:
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@@
 		(in_pos_files yes)
 		(dnp no)
-		(property "Reference" "R401"
+		(property "Reference" "R9"
 			(at 182.88 151.13 0)
 			(show_name no)
@@
 			(project "altera-modular-agilex-5-dc-scm"
 				(path "/6bb9d978-a328-4b30-874b-55170a976185/266bf6db-77fc-4e99-b82f-dd347350f420"
-					(reference "R401")
+					(reference "R9")
 					(unit 1)
 				)
@@
 		(dnp no)
 		(fields_autoplaced yes)
-		(property "Reference" "J100"
+		(property "Reference" "J1"
 			(at 210.185 120.65 0)
 			(show_name no)
@@
 			(project "altera-modular-agilex-5-dc-scm"
 				(path "/6bb9d978-a328-4b30-874b-55170a976185/266bf6db-77fc-4e99-b82f-dd347350f420"
-					(reference "J100")
+					(reference "J1")
 					(unit 4)
 				)
@@
 		(in_pos_files yes)
 		(dnp no)
-		(property "Reference" "#PWR0401"
+		(property "Reference" "#PWR037"
 			(at 172.72 153.67 0)
 			(hide yes)
@@
 			(project "altera-modular-agilex-5-dc-scm"
 				(path "/6bb9d978-a328-4b30-874b-55170a976185/266bf6db-77fc-4e99-b82f-dd347350f420"
-					(reference "#PWR0401")
+					(reference "#PWR037")
 					(unit 1)
 				)

Commit message: [#100501] Add ferrite bead to CLK gen supply, change its decoupling from 1uF to 100nF, rename 20MHz bus to 25MHz
Connections:
- net 20MHz_CLK.+ renamed 25MHz_CLK.+
- net 20MHz_CLK.- renamed 25MHz_CLK.-
Changed lines of the file:
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@@
 		)
 	)
-	(label "20MHz_CLK.+"
+	(label "25MHz_CLK.+"
 		(at 236.22 128.27 0)
 		(effects
@@
 		)
 	)
-	(label "20MHz_CLK.-"
+	(label "25MHz_CLK.-"
 		(at 236.22 130.81 0)
 		(effects
@@
 		)
 	)
-	(hierarchical_label "20MHz_CLK{+ -}"
+	(hierarchical_label "25MHz_CLK{+ -}"
 		(shape input)
 		(at 254 124.46 0)

Commit message: [#100501] Reannotate schematic
Parts:
- renumbered R9 to R3
Changed lines of the file:
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@@
 		(in_pos_files yes)
 		(dnp no)
-		(property "Reference" "R9"
+		(property "Reference" "R3"
 			(at 182.88 151.13 0)
 			(show_name no)
@@
 			(project "altera-modular-agilex-5-dc-scm"
 				(path "/6bb9d978-a328-4b30-874b-55170a976185/266bf6db-77fc-4e99-b82f-dd347350f420"
-					(reference "R9")
+					(reference "R3")
 					(unit 1)
 				)
