File: hs-connector.kicad_sch (KiCad schematic)
At the start: 45 parts, among them J2001 Socket_Samtec_ERF8_2x25_ERF8-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, T2001 Choke_DLW21SN900HQ2L, T2002 Choke_DLW21SN900HQ2L, T2003 Choke_DLW21SN900HQ2L, U2001 SN65MLVD200A

Commit message: [#100282] Move AUX, HPD, CONFIG and AUX_DRV to separate DP_CTRL bus, connect HS connector remaining DP signals
Parts:
- added C2019, C2020: C_1u_0402, antmicro-footprints:C_0402_1005Metric, symbol antmicroCapacitors0402:C_1u_0402
- added U2002: 74AVC4T245_UQFN, antmicro-footprints:UQFN-16-1.8x2.6mm_P0.4mm_Texas_RSV0016A, symbol antmicroLogicTranslatorsLevelShifters:74AVC4T245_UQFN
Connections:
- net +3V3: now also C2020.2, U2002.2 (VCCB)
- net AUX_DRV_IN: now also U2002.13 (2B1)
- net AUX_DRV_OE: now also U2002.15 (1B1)
- net AUX_DRV_OUT: now also U2002.14 (1B2)
- net GND: now also C2019.1, C2020.1, U2002.1 (1~{OE}), U2002.10 (GND), U2002.11 (GND), U2002.16 (2~{OE}), U2002.5 (2DIR)
- net HPD: now also U2002.12 (2B2)
- net AUX+ renamed DP.AUX+
- net AUX- renamed DP.AUX-
- net CFG1 renamed DP.CONFIG1
- new net +1V8: C2019.2, U2002.3 (VCCA), U2002.4 (1DIR)
- new net DP.AUX_DRV_IN: U2002.8 (2A1)
- new net DP.AUX_DRV_OE: U2002.6 (1A1)
- new net DP.AUX_DRV_OUT: U2002.7 (1A2)
- new net DP.HPD: U2002.9 (2A2)
Other:
- moved on the sheet: C2007, C2008, C2017, C2018, D2001, F2001, R2010, R2011, R2012, R2013, R2014, R2015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

Commit message: [#100282] Assign net classes to diff-pairs on HS Connector, improve readability
Connections:
- net ROOTPORT.TX0+: now also C2009.1; no longer C2003.1
- net ROOTPORT.TX0-: now also C2003.1; no longer C2009.1
- net AUX+: now reaches C2011.2, R2003.1, U2001.6 (A)
- net CONN_SFP.RX-: now reaches C2016.2, J2001.47 (37)
- net DP_CONN_TXD.1+: now reaches J2001.10, T2002.2
- net DP_CONN_TXD.1-: now reaches J2001.12, T2002.3
- net DP_CONN_AUX+: now reaches J2001.16, T2003.2
- net DP_CONN_AUX-: now reaches J2001.18, T2003.3
- net CONN_ROOTPORT.TX0+: now reaches J2001.3
- net CONN_ROOTPORT.TX0+: now also C2009.2; no longer C2003.2
- net CONN_SFP.TX+: now reaches C2013.2, J2001.39
- net DP_CONN_TXD.0+: now reaches J2001.4, T2001.2
- net CONN_SFP.TX-: now reaches C2014.2, J2001.41 (31)
- net CONN_SFP.RX+: now reaches C2015.2, J2001.45 (35)
- net CONN_ROOTPORT.TX0-: now reaches J2001.5
- net CONN_ROOTPORT.TX0-: now also C2003.2; no longer C2009.2
- net DP_CONN_TXD.0-: now reaches J2001.6, T2001.3
- net AUX-: now reaches C2012.2, R2004.1, U2001.7 (B)
Other:
- moved on the sheet: C2001, C2007, C2008, C2017, C2018, C2019, C2020, D2001, F2001, R2001, R2002, R2003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

Commit message: [#100282] Fix overlaping graphics, add schematic sheet names on them
Other:
- note added: "High speed connector"
Changed lines of the file:
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@@
 		(company "Altera")
+	)
+	(text "High speed connector"
+		(exclude_from_sim no)
+		(at 203.2 38.1 0)
+		(effects
+			(font
+				(size 4 4)
+				(thickness 0.8)
+				(bold yes)
+			)
+		)
 	)
 	(text_box "1 A -> B\n2 A <- B"
