File: misc.kicad_sch (KiCad schematic)
At the start: 33 parts, among them J2101 Molex_KK_1x2_22-23-2021, Q2101 PJE138K, Q2102 PJE138K, Q2103 PJA3404, SW2101 SW_435441019830_SMD, SW2102 SW_435441019830_SMD, SW2103 SW_435441019830_SMD, SW2104 SW_435441019830_SMD, SW2105 SW_435441019830_SMD

Commit message: [#100282] Add missing schematic sheet names and align them all
Changed lines of the file:
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@@
 	(text "Fan connector"
 		(exclude_from_sim no)
-		(at 203.2 203.2 0)
+		(at 210.82 203.2 0)
 		(effects
 			(font
@@
 	(text "Debug LEDs"
 		(exclude_from_sim no)
-		(at 203.2 114.3 0)
+		(at 210.82 114.3 0)
 		(effects
 			(font
@@
 	(text "Buttons"
 		(exclude_from_sim no)
-		(at 203.2 25.4 0)
+		(at 210.82 25.4 0)
 		(effects
 			(font

Commit message: [#100501] Reannotate schematic
Parts:
- renumbered C2101 to C201, C2102 to C202, C2103 to C203, C2104 to C204, C2105 to C205, D2101 to D2, D2102 to D3, D2103 to D4, D2104 to D5, J2101 to J7, Q2101 to Q4, Q2102 to Q5, Q2103 to Q6, R2101 to R239, R2102 to R240, R2103 to R241, R2104 to R242, R2105 to R243, R2106 to R244, R2107 to R245, R2108 to R246, R2109 to R247, R2110 to R248, R2111 to R249, R2112 to R250, R2113 to R251, R2114 to R252, R2115 to R253, SW2101 to SW1, SW2102 to SW2, SW2103 to SW3, SW2104 to SW4, SW2105 to SW5

Commit message: [#100501] Reannotate schematic
Parts:
- renumbered C201 to C192, C202 to C193, C203 to C194, C204 to C195, C205 to C196, D5 to D10, D2 to D7, D3 to D8, D4 to D9, J7 to J8, Q4 to Q6, Q5 to Q7, Q6 to Q8, R239 to R264, R240 to R265, R241 to R266, R242 to R267, R243 to R268, R244 to R269, R245 to R270, R246 to R271, R247 to R272, R248 to R273, R249 to R274, R250 to R275, R251 to R276, R252 to R277, R253 to R278
