File: mitysom-gts.kicad_sch (KiCad schematic)
At the start: 5 parts, among them J100 Plug_Samtec_SEAM-50-02.0-L-08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

Commit message: [#100501] Reannotate schematic
Parts:
- renumbered C601 to C25, C602 to C26, C603 to C27, C604 to C28, J100 to J1
Changed lines of the file:
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@@
 		(in_pos_files yes)
 		(dnp no)
-		(property "Reference" "C601"
+		(property "Reference" "C25"
 			(at 266.7 110.49 0)
 			(show_name no)
@@
 			(project "altera-modular-agilex-5-dc-scm"
 				(path "/6bb9d978-a328-4b30-874b-55170a976185/82474d56-ea73-4bfa-9277-1decbf47afb2"
-					(reference "C601")
+					(reference "C25")
 					(unit 1)
 				)
@@
 		(in_pos_files yes)
 		(dnp no)
-		(property "Reference" "C602"
+		(property "Reference" "C26"
 			(at 274.32 113.03 0)
 			(show_name no)
@@
 			(project "altera-modular-agilex-5-dc-scm"
 				(path "/6bb9d978-a328-4b30-874b-55170a976185/82474d56-ea73-4bfa-9277-1decbf47afb2"
-					(reference "C602")
+					(reference "C26")
 					(unit 1)
 				)
@@
 		(in_pos_files yes)
 		(dnp no)
-		(property "Reference" "C603"
+		(property "Reference" "C27"
 			(at 266.7 132.08 0)
 			(show_name no)
@@
 			(project "altera-modular-agilex-5-dc-scm"
 				(path "/6bb9d978-a328-4b30-874b-55170a976185/82474d56-ea73-4bfa-9277-1decbf47afb2"
-					(reference "C603")
+					(reference "C27")
 					(unit 1)
 				)
@@
 		(in_pos_files yes)
 		(dnp no)
-		(property "Reference" "C604"
+		(property "Reference" "C28"
 			(at 274.32 134.62 0)
 			(show_name no)
@@
 			(project "altera-modular-agilex-5-dc-scm"
 				(path "/6bb9d978-a328-4b30-874b-55170a976185/82474d56-ea73-4bfa-9277-1decbf47afb2"
-					(reference "C604")
+					(reference "C28")
 					(unit 1)
 				)
@@
 		(dnp no)
 		(fields_autoplaced yes)
-		(property "Reference" "J100"
+		(property "Reference" "J1"
 			(at 213.36 99.06 0)
 			(show_name no)
@@
 			(project "altera-modular-agilex-5-dc-scm"
 				(path "/6bb9d978-a328-4b30-874b-55170a976185/82474d56-ea73-4bfa-9277-1decbf47afb2"
-					(reference "J100")
+					(reference "J1")
 					(unit 3)
 				)

Commit message: [#100595] Update connections according to client request
Parts:
- added C257, C258, C292, C293: C_100n_0402, antmicro-footprints:C_0402_1005Metric, symbol antmicroCapacitors0402:C_100n_0402
Connections:
- net DC_SCM_PCIE.TX1-: now reaches J1.A36 (GTSL1B_RX_CH1_N)
- net DC_SCM_PCIE.TX1+: now reaches J1.A37 (GTSL1B_RX_CH1_P)
- net DC_SCM_PCIE.TX3-: now reaches J1.A40 (GTSL1B_RX_CH3_N)
- net DC_SCM_PCIE.TX3+: now reaches J1.A41 (GTSL1B_RX_CH3_P)
- net DC_SCM_PCIE.TX0-: now reaches J1.G38 (GTSL1B_RX_CH0_N)
- net DC_SCM_PCIE.TX0+: now reaches J1.G39 (GTSL1B_RX_CH0_P)
- net DC_SCM_PCIE.TX2-: now reaches J1.G42 (GTSL1B_RX_CH2_N)
- net DC_SCM_PCIE.TX2+: now reaches J1.G43 (GTSL1B_RX_CH2_P)
- net USBSS1_RX+: now reaches J1.G8 (GTSR4C_RX_CH1_P)
- net USBSS1_RX+: now also C258.2
- net USBSS1_RX-: now reaches J1.G9 (GTSR4C_RX_CH1_N)
- net USBSS1_RX-: now also C293.2
- net USBSS1_TX+: now reaches J1.H10 (GTSR4C_TX_CH1_P)
- net USBSS1_TX+: now also C257.2
- net USBSS1_TX-: now reaches J1.H11 (GTSR4C_TX_CH1_N)
- net USBSS1_TX-: now also C292.2
- net DC_SCM_PCIE.RX2-: now reaches J1.H44 (GTSL1B_TX_CH2_N)
- net DC_SCM_PCIE.RX2+: now reaches J1.H45 (GTSL1B_TX_CH2_P)
- net DC_SCM_PCIE.RX3-: now reaches J1.H48 (GTSL1B_TX_CH3_N)
- net DC_SCM_PCIE.RX3+: now reaches J1.H49 (GTSL1B_TX_CH3_P)
- net DP_HS_CONN.TXD0+ renamed DC_SCM_PCIE.RX0+
- net DP_HS_CONN.TXD0- renamed DC_SCM_PCIE.RX0-
- net DP_HS_CONN.TXD1+ renamed DC_SCM_PCIE.RX1+
- net DP_HS_CONN.TXD1- renamed DC_SCM_PCIE.RX1-
- net USBSS.RX+ renamed USBSS0.RX+
- net USBSS.RX- renamed USBSS0.RX-
- net USBSS.TX+ renamed USBSS0.TX+
- net USBSS.TX- renamed USBSS0.TX-
- net USBSS_RX+ renamed USBSS0_RX+
- net USBSS_RX- renamed USBSS0_RX-
- net USBSS_TX+ renamed USBSS0_TX+
- net USBSS_TX- renamed USBSS0_TX-
- new net USBSS1.RX+: C257.1
- new net USBSS1.RX-: C292.1
- new net USBSS1.TX+: C258.1
- new net USBSS1.TX-: C293.1
- no-connect marks 28 -> 12

Commit message: [#100501] Reannotate schematic
Parts:
- renumbered C257 to C23, C25 to C24, C292 to C25, C258 to C27, C27 to C28, C293 to C29, C28 to C30
Changed lines of the file:
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@@
 		(in_pos_files yes)
 		(dnp no)
-		(property "Reference" "C28"
+		(property "Reference" "C30"
 			(at 274.32 134.62 0)
 			(show_name no)
@@
 			(project "altera-modular-agilex-5-dc-scm"
 				(path "/6bb9d978-a328-4b30-874b-55170a976185/82474d56-ea73-4bfa-9277-1decbf47afb2"
-					(reference "C28")
+					(reference "C30")
 					(unit 1)
 				)
@@
 		(in_pos_files yes)
 		(dnp no)
-		(property "Reference" "C25"
+		(property "Reference" "C24"
 			(at 266.7 110.49 0)
 			(show_name no)
@@
 			(project "altera-modular-agilex-5-dc-scm"
 				(path "/6bb9d978-a328-4b30-874b-55170a976185/82474d56-ea73-4bfa-9277-1decbf47afb2"
-					(reference "C25")
+					(reference "C24")
 					(unit 1)
 				)
@@
 		(in_pos_files yes)
 		(dnp no)
-		(property "Reference" "C27"
+		(property "Reference" "C28"
 			(at 266.7 132.08 0)
 			(show_name no)
@@
 			(project "altera-modular-agilex-5-dc-scm"
 				(path "/6bb9d978-a328-4b30-874b-55170a976185/82474d56-ea73-4bfa-9277-1decbf47afb2"
-					(reference "C27")
+					(reference "C28")
 					(unit 1)
 				)
@@
 		(in_pos_files yes)
 		(dnp no)
-		(property "Reference" "C292"
+		(property "Reference" "C25"
 			(at 152.4 113.03 0)
 			(show_name no)
@@
 			(project "altera-modular-agilex-5-dc-scm"
 				(path "/6bb9d978-a328-4b30-874b-55170a976185/82474d56-ea73-4bfa-9277-1decbf47afb2"
-					(reference "C292")
+					(reference "C25")
 					(unit 1)
 				)
@@
 		(in_pos_files yes)
 		(dnp no)
-		(property "Reference" "C293"
+		(property "Reference" "C29"
 			(at 152.4 134.62 0)
 			(show_name no)
@@
 			(project "altera-modular-agilex-5-dc-scm"
 				(path "/6bb9d978-a328-4b30-874b-55170a976185/82474d56-ea73-4bfa-9277-1decbf47afb2"
-					(reference "C293")
+					(reference "C29")
 					(unit 1)
 				)
@@
 		(in_pos_files yes)
 		(dnp no)
-		(property "Reference" "C258"
+		(property "Reference" "C27"
 			(at 160.02 132.08 0)
 			(show_name no)
@@
 			(project "altera-modular-agilex-5-dc-scm"
 				(path "/6bb9d978-a328-4b30-874b-55170a976185/82474d56-ea73-4bfa-9277-1decbf47afb2"
-					(reference "C258")
+					(reference "C27")
 					(unit 1)
 				)
@@
 		(in_pos_files yes)
 		(dnp no)
-		(property "Reference" "C257"
+		(property "Reference" "C23"
 			(at 160.02 110.49 0)
 			(show_name no)
@@
 			(project "altera-modular-agilex-5-dc-scm"
 				(path "/6bb9d978-a328-4b30-874b-55170a976185/82474d56-ea73-4bfa-9277-1decbf47afb2"
-					(reference "C257")
+					(reference "C23")
 					(unit 1)
 				)
