File: tpm.kicad_sch (KiCad schematic)
At the start: 9 parts, among them J4 PinHeader_2x7_P2mm_Drill0.9mm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, U11 TMUX1574RSVR

Commit message: [#100501] Reannotate schematic
Parts:
- renumbered C83 to C87, R100 to R134, R101 to R135, R102 to R136, R103 to R137, R104 to R138, R105 to R139, U11 to U10
Changed lines of the file:
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@@
 		(in_pos_files yes)
 		(dnp no)
-		(property "Reference" "#PWR0121"
+		(property "Reference" "#PWR0120"
 			(at 218.44 173.99 0)
 			(hide yes)
@@
 			(project "altera-modular-agilex-5-dc-scm"
 				(path "/6bb9d978-a328-4b30-874b-55170a976185/af45e011-8332-484c-9b46-08bd6b2c8877"
-					(reference "#PWR0121")
+					(reference "#PWR0120")
 					(unit 1)
 				)
@@
 		(in_pos_files yes)
 		(dnp no)
-		(property "Reference" "#PWR0125"
+		(property "Reference" "#PWR0124"
 			(at 194.31 182.88 0)
 			(hide yes)
@@
 			(project "altera-modular-agilex-5-dc-scm"
 				(path "/6bb9d978-a328-4b30-874b-55170a976185/af45e011-8332-484c-9b46-08bd6b2c8877"
-					(reference "#PWR0125")
+					(reference "#PWR0124")
 					(unit 1)
 				)
@@
 		(in_pos_files yes)
 		(dnp no)
-		(property "Reference" "R104"
+		(property "Reference" "R138"
 			(at 152.4 170.18 0)
 			(show_name no)
@@
 			(project "altera-modular-agilex-5-dc-scm"
 				(path "/6bb9d978-a328-4b30-874b-55170a976185/af45e011-8332-484c-9b46-08bd6b2c8877"
-					(reference "R104")
+					(reference "R138")
 					(unit 1)
 				)
@@
 		(in_pos_files yes)
 		(dnp no)
-		(property "Reference" "#PWR0124"
+		(property "Reference" "#PWR0123"
 			(at 189.23 182.88 0)
 			(hide yes)
@@
 			(project "altera-modular-agilex-5-dc-scm"
 				(path "/6bb9d978-a328-4b30-874b-55170a976185/af45e011-8332-484c-9b46-08bd6b2c8877"
-					(reference "#PWR0124")
+					(reference "#PWR0123")
 					(unit 1)
 				)
@@
 		(in_pos_files yes)
 		(dnp no)
-		(property "Reference" "R100"
+		(property "Reference" "R134"
 			(at 205.74 132.08 0)
 			(show_name no)
@@
 			(project "altera-modular-agilex-5-dc-scm"
 				(path "/6bb9d978-a328-4b30-874b-55170a976185/af45e011-8332-484c-9b46-08bd6b2c8877"
-					(reference "R100")
+					(reference "R134")
 					(unit 1)
 				)
@@
 		(in_pos_files yes)
 		(dnp yes)
-		(property "Reference" "R103"
+		(property "Reference" "R137"
 			(at 283.21 166.37 0)
 			(show_name no)
@@
 			(project "altera-modular-agilex-5-dc-scm"
 				(path "/6bb9d978-a328-4b30-874b-55170a976185/af45e011-8332-484c-9b46-08bd6b2c8877"
-					(reference "R103")
+					(reference "R137")
 					(unit 1)
 				)
@@
 		(in_pos_files yes)
 		(dnp no)
-		(property "Reference" "R101"
+		(property "Reference" "R135"
 			(at 205.74 142.24 0)
 			(show_name no)
@@
 			(project "altera-modular-agilex-5-dc-scm"
 				(path "/6bb9d978-a328-4b30-874b-55170a976185/af45e011-8332-484c-9b46-08bd6b2c8877"
-					(reference "R101")
+					(reference "R135")
 					(unit 1)
 				)
@@
 		(in_pos_files yes)
 		(dnp no)
-		(property "Reference" "#PWR0126"
+		(property "Reference" "#PWR0125"
 			(at 264.16 182.88 0)
 			(hide yes)
@@
 			(project "altera-modular-agilex-5-dc-scm"
 				(path "/6bb9d978-a328-4b30-874b-55170a976185/af45e011-8332-484c-9b46-08bd6b2c8877"
-					(reference "#PWR0126")
+					(reference "#PWR0125")
 					(unit 1)
 				)
@@
 		(in_pos_files yes)
 		(dnp no)
-		(property "Reference" "U11"
+		(property "Reference" "U10"
 			(at 184.15 124.968 0)
 			(show_name no)
@@
 			(project "altera-modular-agilex-5-dc-scm"
 				(path "/6bb9d978-a328-4b30-874b-55170a976185/af45e011-8332-484c-9b46-08bd6b2c8877"
-					(reference "U11")
+					(reference "U10")
 					(unit 1)
 				)
@@
 		(in_pos_files yes)
 		(dnp no)
-		(property "Reference" "R102"
+		(property "Reference" "R136"
 			(at 283.21 162.56 0)
 			(show_name no)
@@
 			(project "altera-modular-agilex-5-dc-scm"
 				(path "/6bb9d978-a328-4b30-874b-55170a976185/af45e011-8332-484c-9b46-08bd6b2c8877"
-					(reference "R102")
+					(reference "R136")
 					(unit 1)
 				)
@@
 		(in_pos_files yes)
 		(dnp no)
-		(property "Reference" "#PWR0123"
+		(property "Reference" "#PWR0122"
 			(at 161.29 182.88 0)
 			(hide yes)
@@
 			(project "altera-modular-agilex-5-dc-scm"
 				(path "/6bb9d978-a328-4b30-874b-55170a976185/af45e011-8332-484c-9b46-08bd6b2c8877"
-					(reference "#PWR0123")
+					(reference "#PWR0122")
 					(unit 1)
 				)
@@
 		(in_pos_files yes)
 		(dnp no)
-		(property "Reference" "#PWR0122"
+		(property "Reference" "#PWR0121"
 			(at 173.99 182.88 0)
 			(hide yes)
@@
 			(project "altera-modular-agilex-5-dc-scm"
 				(path "/6bb9d978-a328-4b30-874b-55170a976185/af45e011-8332-484c-9b46-08bd6b2c8877"
-					(reference "#PWR0122")
+					(reference "#PWR0121")
 					(unit 1)
 				)
@@
 		(in_pos_files yes)
 		(dnp no)
-		(property "Reference" "R105"
+		(property "Reference" "R139"
 			(at 163.83 175.26 90)
 			(show_name no)
@@
 			(project "altera-modular-agilex-5-dc-scm"
 				(path "/6bb9d978-a328-4b30-874b-55170a976185/af45e011-8332-484c-9b46-08bd6b2c8877"
-					(reference "R105")
+					(reference "R139")
 					(unit 1)
 				)
@@
 		(in_pos_files yes)
 		(dnp no)
-		(property "Reference" "#PWR0120"
+		(property "Reference" "#PWR0119"
 			(at 313.69 162.56 0)
 			(hide yes)
@@
 			(project "altera-modular-agilex-5-dc-scm"
 				(path "/6bb9d978-a328-4b30-874b-55170a976185/af45e011-8332-484c-9b46-08bd6b2c8877"
-					(reference "#PWR0120")
+					(reference "#PWR0119")
 					(unit 1)
 				)
@@
 		(in_pos_files yes)
 		(dnp no)
-		(property "Reference" "C83"
+		(property "Reference" "C87"
 			(at 203.708 174.244 90)
 			(show_name no)
@@
 			(project "altera-modular-agilex-5-dc-scm"
 				(path "/6bb9d978-a328-4b30-874b-55170a976185/af45e011-8332-484c-9b46-08bd6b2c8877"
-					(reference "C83")
+					(reference "C87")
 					(unit 1)
 				)
