File: clk.kicad_sch (KiCad schematic)
At the start: 25 parts, among them U901 SY75602BTWL-TR, U902 SI5338B-B-GM, U903 LMK1C1102DQFT

Commit message: [#100282] Add missing schematic sheet names and align them all
Changed lines of the file:
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@@
 	(text "PCIe clock buffer"
 		(exclude_from_sim no)
-		(at 204.47 41.91 0)
+		(at 210.82 38.1 0)
 		(effects
 			(font
@@
 	(text "Clock generator"
 		(exclude_from_sim no)
-		(at 204.47 172.72 0)
+		(at 210.82 165.1 0)
 		(effects
 			(font

Commit message: [#100501] Reannotate schematic
Parts:
- renumbered C901 to C69, C902 to C70, C903 to C71, C904 to C72, C905 to C73, C906 to C74, C907 to C75, C908 to C76, C909 to C77, C910 to C78, C911 to C79, C912 to C80, C913 to C81, C914 to C82, R901 to R95, R902 to R96, R903 to R97, R904 to R98, R905 to R99, TP901 to TP3, TP902 to TP4, TP903 to TP5, U903 to U10, U901 to U8, U902 to U9

Commit message: [#100501] Add ferrite bead to CLK gen supply, change its decoupling from 1uF to 100nF, rename 20MHz bus to 25MHz
Parts:
- removed C70, C71, C74, C75, C76, C77, C80: C_1u_0402, antmicro-footprints:C_0402_1005Metric, symbol antmicroCapacitors0402:C_1u_0402
- added C259, C260, C261, C262, C263, C264, C265: C_100n_0402, antmicro-footprints:C_0402_1005Metric, symbol antmicroCapacitors0402:C_100n_0402
- added FB4: FB_220Z_2.2A_TDK-MPZ_0603, antmicro-footprints:FB_0603_1608Metric, symbol antmicroFerriteBeadsandChips:FB_220Z_2.2A_TDK-MPZ_0603
Connections:
- net +1V8: now also C265.2, FB4.2; no longer U9.11 (VDDO3), U9.15 (VDDO2), U9.16 (VDDO1), U9.20 (VDDO0), U9.24 (VDD), U9.7 (VDD)
- net 100MHz_CLK+: now also C82.1, U9.13 (CLK2B); no longer C81.1, U9.14 (CLK2A)
- net 100MHz_CLK-: now also C81.1, U9.14 (CLK2A); no longer C82.1, U9.13 (CLK2B)
- net 100MHz_CLK.+: now also C82.2, R97.2; no longer C81.2, R98.2
- net 100MHz_CLK.-: now also C81.2, R98.2; no longer C82.2, R97.2
- net 150MHz_CLK+: now also C73.1, U9.21 (CLK0B); no longer C72.1, U9.22 (CLK0A)
- net 150MHz_CLK-: now also C72.1, U9.22 (CLK0A); no longer C73.1, U9.21 (CLK0B)
- net 150MHz_CLK.+: now also C73.2; no longer C72.2
- net 150MHz_CLK.-: now also C72.2; no longer C73.2
- net 156_25MHz_CLK+: now also C79.1, U9.17 (CLK1B); no longer C78.1, U9.18 (CLK1A)
- net 156_25MHz_CLK-: now also C78.1, U9.18 (CLK1A); no longer C79.1, U9.17 (CLK1B)
- net 156_25MHz_CLK.+: now also C79.2; no longer C78.2
- net 156_25MHz_CLK.-: now also C78.2; no longer C79.2
- net GND: now also C259.1, C260.1, C261.1, C262.1, C263.1, C264.1, C265.1
- net 20MHz_CLK.+ renamed 25MHz_CLK.+
- net 20MHz_CLK.- renamed 25MHz_CLK.-
- new net +1V8_CLK: C259.2, C260.2, C261.2, C262.2, C263.2, C264.2, FB4.1, U9.11 (VDDO3), U9.15 (VDDO2), U9.16 (VDDO1), U9.20 (VDDO0), U9.24 (VDD), U9.7 (VDD)

Commit message: [#100501] Clean ERC
Changed lines of the file:
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@@
 	)
 	(junction
-		(at 182.88 184.15)
-		(diameter 0)
-		(color 0 0 0 0)
-	)
-	(junction
 		(at 160.02 184.15)
 		(diameter 0)
@@
 	)
 	(junction
+		(at 189.23 184.15)
+		(diameter 0)
+		(color 0 0 0 0)
+	)
+	(junction
 		(at 121.92 204.47)
 		(diameter 0)
@@
 	)
 	(junction
+		(at 182.88 184.15)
+		(diameter 0)
+		(color 0 0 0 0)
+	)
+	(junction
 		(at 186.69 204.47)
 		(diameter 0)
@@
 	(wire
 		(pts
+			(xy 190.5 184.15) (xy 189.23 184.15)
+		)
+		(stroke
+			(width 0)
+			(type default)
+		)
+	)
+	(wire
+		(pts
 			(xy 113.03 219.71) (xy 128.27 219.71)
 		)
@@
 	)
 	(label "+1V8_CLK"
-		(at 189.23 184.15 180)
+		(at 187.96 184.15 180)
 		(effects
 			(font
@@
 					(unit 1)
 				)
+			)
+		)
+	)
+	(symbol
+		(lib_id "antmicropower:PWR_FLAG")
+		(at 190.5 184.15 270)
+		(unit 1)
+		(body_style 1)
+		(exclude_from_sim no)
+		(in_bom yes)
+		(on_board yes)
+		(in_pos_files yes)
+		(dnp no)
+		(fields_autoplaced yes)
+		(property "Reference" "#FLG03"
+			(at 192.405 184.15 0)
+			(hide yes)
+			(show_name no)
+			(do_not_autoplace no)
+			(effects
+				(font
+					(size 1.27 1.27)
+				)
+			)
+		)
+		(property "Value" "PWR_FLAG"
+			(at 194.31 184.1499 90)
+			(show_name no)
+			(do_not_autoplace no)
+			(effects
+				(font
+					(size 1.27 1.27)
+				)
+				(justify left)
+			)
+		)
+		(property "Footprint" ""
+			(at 190.5 184.15 0)
+			(hide yes)
+			(show_name no)
+			(do_not_autoplace no)
+			(effects
+				(font
+					(size 1.27 1.27)
+				)
+			)
+		)
+		(property "Datasheet" ""
+			(at 190.5 184.15 0)
+			(hide yes)
+			(show_name no)
+			(do_not_autoplace no)
+			(effects
+				(font
+					(size 1.27 1.27)
+				)
+			)
+		)
+		(property "Description" ""
+			(at 187.96 184.15 0)
+			(hide yes)
+			(show_name no)
+			(do_not_autoplace no)
+			(effects
+				(font
+					(size 1.27 1.27)
+				)
+				(justify left bottom)
+			)
+		)
+		(pin "1"
+		)
+		(instances
+			(project "altera-modular-agilex-5-dc-scm"
+				(path "/6bb9d978-a328-4b30-874b-55170a976185/f9d49440-6457-44a6-96ad-733c78ac7b04"
+					(reference "#FLG03")
+					(unit 1)
+				)

Commit message: [#100501] Reannotate schematic
Parts:
- renumbered C69 to C73, C260 to C74, C259 to C75, C72 to C76, C73 to C77, C261 to C78, C262 to C79, C264 to C80, C263 to C81, C78 to C82, C79 to C83, C265 to C84, C81 to C85, C82 to C86, FB4 to FB1, R95 to R129, R96 to R130, R97 to R131, R98 to R132, R99 to R133, TP3 to TP7, TP4 to TP8, TP5 to TP9, U8 to U7, U9 to U8, U10 to U9

Commit message: [#100501] Perform minor BOM consolidation
Parts:
- C73: value C_1u_0402 -> C_1u_25V_0402; symbol antmicroCapacitors0402:C_1u_0402 -> antmicroCapacitors0402:C_1u_25V_0402; Dielectric (none) -> X5R; MPN C1005X6S1A105K050BC -> GRM155R61E105KE11J; Manufacturer TDK -> Murata; Voltage (none) -> 25V
Changed lines of the file:
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@@
 	)
 	(symbol
-		(lib_id "antmicroCapacitors0402:C_1u_0402")
+		(lib_id "antmicroCapacitors0402:C_1u_25V_0402")
 		(at 187.96 71.12 270)
 		(mirror x)
@@
 			)
 		)
-		(property "Value" "C_1u_0402"
+		(property "Value" "C_1u_25V_0402"
 			(at 177.8 50.8 0)
 			(hide yes)
@@
 			)
 		)
-		(property "Datasheet" "https://product.tdk.com/en/search/capacitor/ceramic/mlcc/info?part_no=C1005X6S1A105K050BC"
+		(property "Datasheet" "https://www.murata.com/products/productdetail?partno=GRM155R61E105KE11%23"
 			(at 172.72 50.8 0)
 			(hide yes)
@@
 			)
 		)
-		(property "Description" "SMD Multilayer Ceramic Capacitor, 1 µF, 10 V, 0402 [1005 Metric], ± 10%, X6S, C"
+		(property "Description" "SMD Multilayer Ceramic Capacitor, 1 µF, 25 V, 0402 [1005 Metric], ± 10%, X5R, GRM Series"
 			(at 154.94 50.8 0)
 			(hide yes)
@@
 			)
 		)
-		(property "MPN" "C1005X6S1A105K050BC"
+		(property "MPN" "GRM155R61E105KE11J"
 			(at 170.18 50.8 0)
 			(hide yes)
@@
 			)
 		)
-		(property "Manufacturer" "TDK"
+		(property "Manufacturer" "Murata"
 			(at 167.64 50.8 0)
 			(hide yes)
@@
 			)
 		)
-		(property "Voltage" ""
+		(property "Voltage" "25V"
 			(at 160.02 50.8 0)
 			(hide yes)
@@
 			)
 		)
-		(property "Dielectric" ""
+		(property "Dielectric" "X5R"
 			(at 157.48 50.8 0)
 			(hide yes)
