File: clk.kicad_sch (KiCad schematic)
At the start: 39 parts, among them U46 SY75602BTWL-TR, U47 DSC557-0344FI0T, U7 SY75604BTWL-TR, U8 SI5338B-B-GM, U9 LMK1C1102DQFT

Commit message: [#100687] Update power label
Parts:
- removed U7: SY75604BTWL-TR, antmicro-footprints:VQFN-16-1EP_3x3mm_P0.5mm_EP1.68x1.68mm, symbol antmicroClockTimingClockGeneratorsPLLsFrequencySynthesizers:SY75604BTWL-TR_1
- added U7: SY75604BTWL-TR, antmicro-footprints:VQFN-16-1EP_3x3mm_P0.5mm_EP1.68x1.68mm, symbol antmicroClockTimingClockGeneratorsPLLsFrequencySynthesizers:SY75604BTWL-TR
Connections:
- net +3V3: now also U7.13 (VDD), U7.16 (OE3b)
- net DC_SCM_CLK.CLK+: now also U7.1 (IN_P)
- net DC_SCM_CLK.CLK-: now also U7.2 (IN_N)
- net GND: now also U7.12 (OE2b), U7.3 (OE0b), U7.6 (OE1b), U7.9 (GND)
- net PCIEx4_CLK.CLK+: now also U7.10 (OUT2_P)
- net PCIEx4_CLK.CLK-: now also U7.11 (OUT2_N)
- net SOM_CLK+: now also U7.7 (OUT1_P)
- net SOM_CLK-: now also U7.8 (OUT1_N)
- net USB_CLK.CLK+: now also U7.4 (OUT0_P)
- net USB_CLK.CLK-: now also U7.5 (OUT0_N)
Changed lines of the file:
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@@
 	)
 	(symbol
+		(lib_id "antmicroClockTimingClockGeneratorsPLLsFrequencySynthesizers:SY75604BTWL-TR")
+		(at 267.97 77.47 0)
+		(unit 1)
+		(body_style 1)
+		(exclude_from_sim no)
+		(in_bom yes)
+		(on_board yes)
+		(in_pos_files yes)
+		(dnp no)
+		(fields_autoplaced yes)
+		(property "Reference" "U7"
+			(at 278.13 69.85 0)
+			(show_name no)
+			(do_not_autoplace no)
+			(effects
+				(font
+					(size 1.27 1.27)
+					(thickness 0.15)
+				)
+			)
+		)
+		(property "Value" "SY75604BTWL-TR"
+			(at 300.99 85.09 0)
+			(hide yes)
+			(show_name no)
+			(do_not_autoplace no)
+			(effects
+				(font
+					(size 1.27 1.27)
+					(thickness 0.15)
+				)
+				(justify left bottom)
+			)
+		)
+		(property "Footprint" "antmicro-footprints:VQFN-16-1EP_3x3mm_P0.5mm_EP1.68x1.68mm"
+			(at 300.99 87.63 0)
+			(hide yes)
+			(show_name no)
+			(do_not_autoplace no)
+			(effects
+				(font
+					(size 1.27 1.27)
+					(thickness 0.15)
+				)
+				(justify left bottom)
+			)
+		)
+		(property "Datasheet" "https://ww1.microchip.com/downloads/aemDocuments/documents/TCG/ProductDocuments/DataSheets/SY75602A-02B-03A-03B-04A-04B-2-4-Outputs-Ultra-Low-Additive-Jitter-PCIe-1-2-3-4-5-6-Clock-Buffer-DS20006508.pdf"
+			(at 300.99 90.17 0)
+			(hide yes)
+			(show_name no)
+			(do_not_autoplace no)
+			(effects
+				(font
+					(size 1.27 1.27)
+					(thickness 0.15)
+				)
+				(justify left bottom)
+			)
+		)
+		(property "Description" "PCIe CLK BUFFER 1:4 250MHZ, small package VQFN-16"
+			(at 300.99 102.87 0)
+			(hide yes)
+			(show_name no)
+			(do_not_autoplace no)
+			(effects
+				(font
+					(size 1.27 1.27)
+					(thickness 0.15)
+				)
+				(justify left bottom)
+			)
+		)
+		(property "Manufacturer" "Microchip Technology"
+			(at 300.99 95.25 0)
+			(hide yes)
+			(show_name no)
+			(do_not_autoplace no)
+			(effects
+				(font
+					(size 1.27 1.27)
+					(thickness 0.15)
+				)
+				(justify left bottom)
+			)
+		)
+		(property "MPN" "SY75604BTWL-TR"
+			(at 278.13 72.39 0)
+			(show_name no)
+			(do_not_autoplace no)
+			(effects
+				(font
+					(size 1.27 1.27)
+					(thickness 0.15)
+				)
+			)
+		)
+		(property "Author" "Antmicro"
+			(at 300.99 97.79 0)
+			(hide yes)
+			(show_name no)
+			(do_not_autoplace no)
+			(effects
+				(font
+					(size 1.27 1.27)
+					(thickness 0.15)
+				)
+				(justify left bottom)
+			)
+		)
+		(property "License" "Apache-2.0"
+			(at 300.99 100.33 0)
+			(hide yes)
+			(show_name no)
+			(do_not_autoplace no)
+			(effects
+				(font
+					(size 1.27 1.27)
+					(thickness 0.15)
+				)
+				(justify left bottom)
+			)
+		)
+		(pin "6"
+		)
+		(pin "15"
+		)
+		(pin "11"
+		)
+		(pin "12"
+		)
+		(pin "10"
+		)
+		(pin "13"
+		)
+		(pin "9"
+		)
+		(pin "7"
+		)
+		(pin "1"
+		)
+		(pin "4"
+		)
+		(pin "8"
+		)
+		(pin "5"
+		)
+		(pin "2"
+		)
+		(pin "14"
+		)
+		(pin "3"
+		)
+		(pin "16"
+		)
+		(instances
+			(project "altera-modular-agilex-5-dc-scm"
+				(path "/6bb9d978-a328-4b30-874b-55170a976185/f9d49440-6457-44a6-96ad-733c78ac7b04"
+					(reference "U7")
+					(unit 1)
+				)
+			)
+		)
+	)
+	(symbol
 		(lib_id "antmicroCapacitors0402:C_100n_0402")
 		(at 252.73 217.17 0)
@@
 					(unit 1)
 				)
-			)
-		)
-	)
-	(symbol
-		(lib_id "antmicroClockTimingClockGeneratorsPLLsFrequencySynthesizers:SY75604BTWL-TR_1")
-		(at 267.97 77.47 0)
-		(unit 1)
-		(body_style 1)
-		(exclude_from_sim no)
-		(in_bom yes)
-		(on_board yes)
-		(in_pos_files yes)
-		(dnp no)
-		(fields_autoplaced yes)
-		(property "Reference" "U7"
-			(at 278.13 69.85 0)
-			(show_name no)
-			(do_not_autoplace no)
-			(effects
-				(font
-					(size 1.27 1.27)
-					(thickness 0.15)
-				)
-			)
-		)
-		(property "Value" "SY75604BTWL-TR"
-			(at 300.99 85.09 0)
-			(hide yes)
-			(show_name no)
-			(do_not_autoplace no)
-			(effects
-				(font
-					(size 1.27 1.27)
-					(thickness 0.15)
-				)
-				(justify left bottom)
-			)
-		)
-		(property "Footprint" "antmicro-footprints:VQFN-16-1EP_3x3mm_P0.5mm_EP1.68x1.68mm"
-			(at 300.99 87.63 0)
-			(hide yes)
-			(show_name no)
-			(do_not_autoplace no)
-			(effects
-				(font
-					(size 1.27 1.27)
-					(thickness 0.15)
-				)
-				(justify left bottom)
-			)
-		)
-		(property "Datasheet" "https://ww1.microchip.com/downloads/aemDocuments/documents/TCG/ProductDocuments/DataSheets/SY75602A-02B-03A-03B-04A-04B-2-4-Outputs-Ultra-Low-Additive-Jitter-PCIe-1-2-3-4-5-6-Clock-Buffer-DS20006508.pdf"
-			(at 300.99 90.17 0)
-			(hide yes)
-			(show_name no)
-			(do_not_autoplace no)
-			(effects
-				(font
-					(size 1.27 1.27)
-					(thickness 0.15)
-				)
-				(justify left bottom)
-			)
-		)
-		(property "Description" "PCIe CLK BUFFER 1:4 250MHZ, small package VQFN-16"
-			(at 300.99 102.87 0)
-			(hide yes)
-			(show_name no)
-			(do_not_autoplace no)
-			(effects
-				(font
-					(size 1.27 1.27)
-					(thickness 0.15)
-				)
-				(justify left bottom)
-			)
-		)
-		(property "Manufacturer" "Microchip Technology"
-			(at 300.99 95.25 0)
-			(hide yes)
-			(show_name no)
-			(do_not_autoplace no)
-			(effects
-				(font
-					(size 1.27 1.27)
-					(thickness 0.15)
-				)
-				(justify left bottom)
-			)
-		)
-		(property "MPN" "SY75604BTWL-TR"
-			(at 278.13 72.39 0)
-			(show_name no)
-			(do_not_autoplace no)
-			(effects
-				(font
-					(size 1.27 1.27)
-					(thickness 0.15)
-				)
-			)
-		)
-		(property "Author" "Antmicro"
-			(at 300.99 97.79 0)
-			(hide yes)
-			(show_name no)
-			(do_not_autoplace no)
-			(effects
-				(font
-					(size 1.27 1.27)
-					(thickness 0.15)
-				)
-				(justify left bottom)
-			)
-		)
-		(property "License" "Apache-2.0"
-			(at 300.99 100.33 0)
-			(hide yes)
-			(show_name no)
-			(do_not_autoplace no)
-			(effects
-				(font
-					(size 1.27 1.27)
-					(thickness 0.15)
-				)
-				(justify left bottom)
-			)
-		)
-		(pin "9"
-		)
-		(pin "14"
-		)
-		(pin "11"
-		)
-		(pin "15"
-		)
-		(pin "10"
-		)
-		(pin "12"
-		)
-		(pin "7"
-		)
-		(pin "2"
-		)
-		(pin "1"
-		)
-		(pin "4"
-		)
-		(pin "5"
-		)
-		(pin "3"
-		)
-		(pin "6"
-		)
-		(pin "8"
-		)
-		(pin "16"
-		)
-		(pin "13"
-		)
-		(instances
-			(project "altera-modular-agilex-5-dc-scm"
-				(path "/6bb9d978-a328-4b30-874b-55170a976185/f9d49440-6457-44a6-96ad-733c78ac7b04"
-					(reference "U7")
-					(unit 1)
-				)

Commit message: [#100687] Update I2C connections
Parts:
- U7: footprint antmicro-footprints:VQFN-16-1EP_3x3mm_P0.5mm_EP1.68x1.68mm -> antmicro-footprints:VQFN-16-1EP_3x3mm_P0.5mm_EP1.1x1.1mm
Changed lines of the file:
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@@
 			)
 		)
-		(property "Footprint" "antmicro-footprints:VQFN-16-1EP_3x3mm_P0.5mm_EP1.68x1.68mm"
+		(property "Footprint" "antmicro-footprints:VQFN-16-1EP_3x3mm_P0.5mm_EP1.1x1.1mm"
 			(at 300.99 87.63 0)
 			(hide yes)
