File: front-panel-usb.kicad_sch (KiCad schematic)
At the start: 89 parts, among them J10 USB-C_Kycon_KUSBX-SL2-CS1N24-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, J11 USB-C_Kycon_KUSBX-SL2-CS1N24-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, J9 USB-C_Kycon_KUSBX-SL2-CS1N24-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, Q9 PJE138K, U26 AP22615B_TSOT26, U27 FUSB303B, U28 TPD4E05U06QDQARQ1, U29 TPD4E05U06QDQARQ1, U30 AP22615B_TSOT26, U31 HD3SS3220RNH, U32 TPD4E05U06QDQARQ1, U33 74LVC06ABQ, U34 TPD4E05U06QDQARQ1, U35 TPD4E05U06QDQARQ1, U36 74AUP2G132

Commit message: [#100501] Perform minor BOM consolidation
Parts:
- C197, C200, C203, C207, C208, C209, C215: value C_1u_0402 -> C_1u_25V_0402; symbol antmicroCapacitors0402:C_1u_0402 -> antmicroCapacitors0402:C_1u_25V_0402; Dielectric (none) -> X5R; MPN C1005X6S1A105K050BC -> GRM155R61E105KE11J; Manufacturer TDK -> Murata; Voltage (none) -> 25V
Changed lines of the file:
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@@
 	)
 	(symbol
-		(lib_id "antmicroCapacitors0402:C_1u_0402")
+		(lib_id "antmicroCapacitors0402:C_1u_25V_0402")
 		(at 38.1 185.42 270)
 		(mirror x)
@@
 			)
 		)
-		(property "Value" "C_1u_0402"
+		(property "Value" "C_1u_25V_0402"
 			(at 27.94 165.1 0)
 			(hide yes)
@@
 			)
 		)
-		(property "Datasheet" "https://product.tdk.com/en/search/capacitor/ceramic/mlcc/info?part_no=C1005X6S1A105K050BC"
+		(property "Datasheet" "https://www.murata.com/products/productdetail?partno=GRM155R61E105KE11%23"
 			(at 22.86 165.1 0)
 			(hide yes)
@@
 			)
 		)
-		(property "Description" "SMD Multilayer Ceramic Capacitor, 1 µF, 10 V, 0402 [1005 Metric], ± 10%, X6S, C"
+		(property "Description" "SMD Multilayer Ceramic Capacitor, 1 µF, 25 V, 0402 [1005 Metric], ± 10%, X5R, GRM Series"
 			(at 5.08 165.1 0)
 			(hide yes)
@@
 			)
 		)
-		(property "MPN" "C1005X6S1A105K050BC"
+		(property "MPN" "GRM155R61E105KE11J"
 			(at 20.32 165.1 0)
 			(hide yes)
@@
 			)
 		)
-		(property "Manufacturer" "TDK"
+		(property "Manufacturer" "Murata"
 			(at 17.78 165.1 0)
 			(hide yes)
@@
 			)
 		)
-		(property "Voltage" ""
+		(property "Voltage" "25V"
 			(at 10.16 165.1 0)
 			(hide yes)
@@
 			)
 		)
-		(property "Dielectric" ""
+		(property "Dielectric" "X5R"
 			(at 7.62 165.1 0)
 			(hide yes)
@@
 	)
 	(symbol
-		(lib_id "antmicroCapacitors0402:C_1u_0402")
+		(lib_id "antmicroCapacitors0402:C_1u_25V_0402")
 		(at 236.22 34.29 270)
 		(mirror x)
@@
 			)
 		)
-		(property "Value" "C_1u_0402"
+		(property "Value" "C_1u_25V_0402"
 			(at 226.06 13.97 0)
 			(hide yes)
@@
 			)
 		)
-		(property "Datasheet" "https://product.tdk.com/en/search/capacitor/ceramic/mlcc/info?part_no=C1005X6S1A105K050BC"
+		(property "Datasheet" "https://www.murata.com/products/productdetail?partno=GRM155R61E105KE11%23"
 			(at 220.98 13.97 0)
 			(hide yes)
@@
 			)
 		)
-		(property "Description" "SMD Multilayer Ceramic Capacitor, 1 µF, 10 V, 0402 [1005 Metric], ± 10%, X6S, C"
+		(property "Description" "SMD Multilayer Ceramic Capacitor, 1 µF, 25 V, 0402 [1005 Metric], ± 10%, X5R, GRM Series"
 			(at 203.2 13.97 0)
 			(hide yes)
@@
 			)
 		)
-		(property "MPN" "C1005X6S1A105K050BC"
+		(property "MPN" "GRM155R61E105KE11J"
 			(at 218.44 13.97 0)
 			(hide yes)
@@
 			)
 		)
-		(property "Manufacturer" "TDK"
+		(property "Manufacturer" "Murata"
 			(at 215.9 13.97 0)
 			(hide yes)
@@
 			)
 		)
-		(property "Voltage" ""
+		(property "Voltage" "25V"
 			(at 208.28 13.97 0)
 			(hide yes)
@@
 			)
 		)
-		(property "Dielectric" ""
+		(property "Dielectric" "X5R"
 			(at 205.74 13.97 0)
 			(hide yes)
@@
 	)
 	(symbol
-		(lib_id "antmicroCapacitors0402:C_1u_0402")
+		(lib_id "antmicroCapacitors0402:C_1u_25V_0402")
 		(at 214.63 149.86 90)
 		(unit 1)
@@
 			)
 		)
-		(property "Value" "C_1u_0402"
+		(property "Value" "C_1u_25V_0402"
 			(at 224.79 129.54 0)
 			(hide yes)
@@
 			)
 		)
-		(property "Datasheet" "https://product.tdk.com/en/search/capacitor/ceramic/mlcc/info?part_no=C1005X6S1A105K050BC"
+		(property "Datasheet" "https://www.murata.com/products/productdetail?partno=GRM155R61E105KE11%23"
 			(at 229.87 129.54 0)
 			(hide yes)
@@
 			)
 		)
-		(property "Description" "SMD Multilayer Ceramic Capacitor, 1 µF, 10 V, 0402 [1005 Metric], ± 10%, X6S, C"
+		(property "Description" "SMD Multilayer Ceramic Capacitor, 1 µF, 25 V, 0402 [1005 Metric], ± 10%, X5R, GRM Series"
 			(at 247.65 129.54 0)
 			(hide yes)
@@
 			)
 		)
-		(property "MPN" "C1005X6S1A105K050BC"
+		(property "MPN" "GRM155R61E105KE11J"
 			(at 232.41 129.54 0)
 			(hide yes)
@@
 			)
 		)
-		(property "Manufacturer" "TDK"
+		(property "Manufacturer" "Murata"
 			(at 234.95 129.54 0)
 			(hide yes)
@@
 			)
 		)
-		(property "Voltage" ""
+		(property "Voltage" "25V"
 			(at 242.57 129.54 0)
 			(hide yes)
@@
 			)
 		)
-		(property "Dielectric" ""
+		(property "Dielectric" "X5R"
 			(at 245.11 129.54 0)
 			(hide yes)
@@
 	)
 	(symbol
-		(lib_id "antmicroCapacitors0402:C_1u_0402")
+		(lib_id "antmicroCapacitors0402:C_1u_25V_0402")
 		(at 271.78 62.23 270)
 		(mirror x)
@@
 			)
 		)
-		(property "Value" "C_1u_0402"
+		(property "Value" "C_1u_25V_0402"
 			(at 261.62 41.91 0)
 			(hide yes)
@@
 			)
 		)
-		(property "Datasheet" "https://product.tdk.com/en/search/capacitor/ceramic/mlcc/info?part_no=C1005X6S1A105K050BC"
+		(property "Datasheet" "https://www.murata.com/products/productdetail?partno=GRM155R61E105KE11%23"
 			(at 256.54 41.91 0)
 			(hide yes)
@@
 			)
 		)
-		(property "Description" "SMD Multilayer Ceramic Capacitor, 1 µF, 10 V, 0402 [1005 Metric], ± 10%, X6S, C"
+		(property "Description" "SMD Multilayer Ceramic Capacitor, 1 µF, 25 V, 0402 [1005 Metric], ± 10%, X5R, GRM Series"
 			(at 238.76 41.91 0)
 			(hide yes)
@@
 			)
 		)
-		(property "MPN" "C1005X6S1A105K050BC"
+		(property "MPN" "GRM155R61E105KE11J"
 			(at 254 41.91 0)
 			(hide yes)
@@
 			)
 		)
-		(property "Manufacturer" "TDK"
+		(property "Manufacturer" "Murata"
 			(at 251.46 41.91 0)
 			(hide yes)
@@
 			)
 		)
-		(property "Voltage" ""
+		(property "Voltage" "25V"
 			(at 243.84 41.91 0)
 			(hide yes)
@@
 			)
 		)
-		(property "Dielectric" ""
+		(property "Dielectric" "X5R"
 			(at 241.3 41.91 0)
 			(hide yes)
@@
 	)
 	(symbol
-		(lib_id "antmicroCapacitors0402:C_1u_0402")
+		(lib_id "antmicroCapacitors0402:C_1u_25V_0402")
 		(at 196.85 149.86 270)
 		(mirror x)
@@
 			)
 		)
-		(property "Value" "C_1u_0402"
+		(property "Value" "C_1u_25V_0402"
 			(at 186.69 129.54 0)
 			(hide yes)
@@
 			)
 		)
-		(property "Datasheet" "https://product.tdk.com/en/search/capacitor/ceramic/mlcc/info?part_no=C1005X6S1A105K050BC"
+		(property "Datasheet" "https://www.murata.com/products/productdetail?partno=GRM155R61E105KE11%23"
 			(at 181.61 129.54 0)
 			(hide yes)
@@
 			)
 		)
-		(property "Description" "SMD Multilayer Ceramic Capacitor, 1 µF, 10 V, 0402 [1005 Metric], ± 10%, X6S, C"
+		(property "Description" "SMD Multilayer Ceramic Capacitor, 1 µF, 25 V, 0402 [1005 Metric], ± 10%, X5R, GRM Series"
 			(at 163.83 129.54 0)
 			(hide yes)
@@
 			)
 		)
-		(property "MPN" "C1005X6S1A105K050BC"
+		(property "MPN" "GRM155R61E105KE11J"
 			(at 179.07 129.54 0)
 			(hide yes)
@@
 			)
 		)
-		(property "Manufacturer" "TDK"
+		(property "Manufacturer" "Murata"
 			(at 176.53 129.54 0)
 			(hide yes)
@@
 			)
 		)
-		(property "Voltage" ""
+		(property "Voltage" "25V"
 			(at 168.91 129.54 0)
 			(hide yes)
@@
 			)
 		)
-		(property "Dielectric" ""
+		(property "Dielectric" "X5R"
 			(at 166.37 129.54 0)
 			(hide yes)
@@
 	)
 	(symbol
-		(lib_id "antmicroCapacitors0402:C_1u_0402")
+		(lib_id "antmicroCapacitors0402:C_1u_25V_0402")
 		(at 237.49 252.73 270)
 		(mirror x)
@@
 			)
 		)
-		(property "Value" "C_1u_0402"
+		(property "Value" "C_1u_25V_0402"
 			(at 227.33 232.41 0)
 			(hide yes)
@@
 			)
 		)
-		(property "Datasheet" "https://product.tdk.com/en/search/capacitor/ceramic/mlcc/info?part_no=C1005X6S1A105K050BC"
+		(property "Datasheet" "https://www.murata.com/products/productdetail?partno=GRM155R61E105KE11%23"
 			(at 222.25 232.41 0)
 			(hide yes)
@@
 			)
 		)
-		(property "Description" "SMD Multilayer Ceramic Capacitor, 1 µF, 10 V, 0402 [1005 Metric], ± 10%, X6S, C"
+		(property "Description" "SMD Multilayer Ceramic Capacitor, 1 µF, 25 V, 0402 [1005 Metric], ± 10%, X5R, GRM Series"
 			(at 204.47 232.41 0)
 			(hide yes)
@@
 			)
 		)
-		(property "MPN" "C1005X6S1A105K050BC"
+		(property "MPN" "GRM155R61E105KE11J"
 			(at 219.71 232.41 0)
 			(hide yes)
@@
 			)
 		)
-		(property "Manufacturer" "TDK"
+		(property "Manufacturer" "Murata"
 			(at 217.17 232.41 0)
 			(hide yes)
@@
 			)
 		)
-		(property "Voltage" ""
+		(property "Voltage" "25V"
 			(at 209.55 232.41 0)
 			(hide yes)
@@
 			)
 		)
-		(property "Dielectric" ""
+		(property "Dielectric" "X5R"
 			(at 207.01 232.41 0)
 			(hide yes)
@@
 	)
 	(symbol
-		(lib_id "antmicroCapacitors0402:C_1u_0402")
+		(lib_id "antmicroCapacitors0402:C_1u_25V_0402")
 		(at 289.56 128.27 90)
 		(unit 1)
@@
 			)
 		)
-		(property "Value" "C_1u_0402"
+		(property "Value" "C_1u_25V_0402"
 			(at 299.72 107.95 0)
 			(hide yes)
@@
 			)
 		)
-		(property "Datasheet" "https://product.tdk.com/en/search/capacitor/ceramic/mlcc/info?part_no=C1005X6S1A105K050BC"
+		(property "Datasheet" "https://www.murata.com/products/productdetail?partno=GRM155R61E105KE11%23"
 			(at 304.8 107.95 0)
 			(hide yes)
@@
 			)
 		)
-		(property "Description" "SMD Multilayer Ceramic Capacitor, 1 µF, 10 V, 0402 [1005 Metric], ± 10%, X6S, C"
+		(property "Description" "SMD Multilayer Ceramic Capacitor, 1 µF, 25 V, 0402 [1005 Metric], ± 10%, X5R, GRM Series"
 			(at 322.58 107.95 0)
 			(hide yes)
@@
 			)
 		)
-		(property "MPN" "C1005X6S1A105K050BC"
+		(property "MPN" "GRM155R61E105KE11J"
 			(at 307.34 107.95 0)
 			(hide yes)
@@
 			)
 		)
-		(property "Manufacturer" "TDK"
+		(property "Manufacturer" "Murata"
 			(at 309.88 107.95 0)
 			(hide yes)
@@
 			)
 		)
-		(property "Voltage" ""
+		(property "Voltage" "25V"
 			(at 317.5 107.95 0)
 			(hide yes)
@@
 			)
 		)
-		(property "Dielectric" ""
+		(property "Dielectric" "X5R"
 			(at 320.04 107.95 0)
 			(hide yes)
