File: usb-controller.kicad_sch (KiCad schematic)
At the start: 63 parts, among them J14 Tag-Connect_TC2050-IDC-NL_2x5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, Q2 PJE138K, Q3 PJE138K, U20 W25Q80DV_USON, U48 UPD720201K8-701-BAC-A, Y7 Resonator_24MHz_ECX-1247

Commit message: [#100501] Reannotate schematic
Parts:
- renumbered C266 to C109, C268 to C110, C269 to C111, C270 to C112, C272 to C113, C273 to C114, C274 to C115, C277 to C116, C278 to C117, C279 to C118, C280 to C119, C281 to C120, C283 to C121, C285 to C122, C287 to C123, C288 to C124, C289 to C125, C286 to C126, C284 to C127, C282 to C128, C127 to C129, C128 to C130, C275 to C131, C276 to C132, C129 to C133, C267 to C134, C271 to C135, D18 to D5, FB5 to FB2, J14 to J6, Q2 to Q4, Q3 to Q5, R371 to R187, R370 to R188, R364 to R189, R153 to R190, R353 to R191, R155 to R192, R157 to R193, R163 to R194, R162 to R195, R161 to R196, R361 to R197, R160 to R198, R357 to R199, R166 to R200, R368 to R201, R369 to R202, R358 to R203, R219 to R204, R220 to R205, R359 to R206, R360 to R207, R165 to R208, R362 to R209, R363 to R210, R367 to R211, TP32 to TP24, TP33 to TP25, TP34 to TP26, U48 to U18, U20 to U19, Y7 to Y1

Commit message: [#100501] Perform minor BOM consolidation
Parts:
- C109, C125, C129: value C_1u_10V_X7R_0402 -> C_1u_25V_0402; symbol antmicroCapacitors0402:C_1u_10V_X7R_0402 -> antmicroCapacitors0402:C_1u_25V_0402; Dielectric X7R -> X5R; MPN GRM155Z71A105KE01D -> GRM155R61E105KE11J; Voltage 10V -> 25V
- C110, C111, C112, C113, C114, C115, C116, C117, C118, C119, C120, C121, C122, C123, C124, C127, C128, C131, C132, C133: value C_100n_16V_X7R_0402 -> C_100n_0402; symbol antmicroCapacitors0402:C_100n_16V_X7R_0402 -> antmicroCapacitors0402:C_100n_0402; Dielectric X7R -> X5R; MPN C0402C104J4RAC7411 -> GRM155R61H104KE14D; Manufacturer KEMET -> Murata; Voltage 16V -> 50V
- C126: value C_10u_6.3V_0402 -> C_10u_0402; symbol antmicroCapacitors0402:C_10u_6.3V_0402 -> antmicroCapacitors0402:C_10u_0402; MPN GRM155R60J106ME15D -> CC0402MRX5R5BB106; Manufacturer Murata -> YAGEO
