File: front-panel-dp.kicad_sch (KiCad schematic)
At the start: 31 parts, among them J14 DisplayPort-Mini_Pulse_E9320-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, T1 Choke_DLW21SN900HQ2L, T2 Choke_DLW21SN900HQ2L, T3 Choke_DLW21SN900HQ2L, U43 TPD4E05U06QDQARQ1, U44 SN65MLVD200A, U45 TPD4E05U06QDQARQ1

Commit message: [#100707] Connect power and low speed signals
Connections:
- net DP.CONFIG1: now also U45.1, U45.10
- no-connect marks 6 -> 5
Changed lines of the file:
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@@
-	)
-	(no_connect
-		(at 342.9 134.62)
 	)
 	(no_connect
@@
 	(wire
 		(pts
+			(xy 325.0754 131.9295) (xy 337.7754 131.9295)
+		)
+		(stroke
+			(width 0)
+			(type default)
+		)
+	)
+	(wire
+		(pts
 			(xy 137.16 100.33) (xy 137.16 101.6)
 		)
@@
 		(pts
 			(xy 260.35 99.06) (xy 260.35 97.79)
+		)
+		(stroke
+			(width 0)
+			(type default)
+		)
+	)
+	(wire
+		(pts
+			(xy 326.39 134.62) (xy 342.9 134.62)
 		)
 		(stroke
@@
 	)
 	(label "DP.CONFIG1"
+		(at 337.7754 131.9295 180)
+		(effects
+			(font
+				(size 1.27 1.27)
+			)
+			(justify right bottom)
+		)
+	)
+	(label "DP.CONFIG1"
 		(at 316.23 130.81 180)
 		(effects
@@
 	(label "DPCONN_AUX-"
 		(at 326.39 142.24 0)
+		(effects
+			(font
+				(size 1.27 1.27)
+			)
+			(justify left bottom)
+		)
+	)
+	(label "DP.CONFIG1"
+		(at 326.39 134.62 0)
 		(effects
 			(font
@@
 			(justify left bottom)
 		)
-		(property "Net Class" "100Ohm-diff"
+		(property "Netclass" "100Ohm-diff"
 			(at 212.7885 90.17 0)
 			(show_name no)
@@
 			(justify left bottom)
 		)
-		(property "Net Class" "100Ohm-diff"
+		(property "Netclass" "100Ohm-diff"
 			(at 168.148 92.71 0)
 			(show_name no)
@@
 			(justify left bottom)
 		)
-		(property "Net Class" "100Ohm-diff"
+		(property "Netclass" "100Ohm-diff"
 			(at 259.7785 90.17 0)
 			(show_name no)
@@
 			(justify left bottom)
 		)
-		(property "Net Class" "100Ohm-diff"
+		(property "Netclass" "100Ohm-diff"
 			(at 155.6385 120.65 0)
 			(show_name no)

Commit message: [#101340] Add flash sockets
Changed lines of the file:
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@@
-	(wire
-		(pts
-			(xy 325.0754 131.9295) (xy 337.7754 131.9295)
-		)
-		(stroke
-			(width 0)
-			(type default)
-		)
-	)
 	(wire
 		(pts
@@
 		)
 	)
-	(label "DP.CONFIG1"
-		(at 337.7754 131.9295 180)
-		(effects
-			(font
-				(size 1.27 1.27)
-			)
-			(justify right bottom)
-		)
-	)

Commit message: [#101340] Use one MPN for Schottky diodes
Parts:
- D26: value RB521S30T1G -> PMEG3010CEJ,115; footprint antmicro-footprints:SOD-523 -> antmicro-footprints:D_SOD-323F; symbol antmicroDiodesRectifiersSingle:RB521S30T1G -> antmicroDiodesRectifiersSingle:PMEG3010CEJ,115; MPN RB521S30T1G -> PMEG3010CEJ,115; Manufacturer ON Semiconductor -> Nexperia
Changed lines of the file:
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@@
 	)
 	(symbol
-		(lib_id "antmicroDiodesRectifiersSingle:RB521S30T1G")
+		(lib_id "antmicroDiodesRectifiersSingle:PMEG3010CEJ,115")
 		(at 240.03 138.43 180)
 		(unit 1)
@@
 		(in_pos_files yes)
 		(dnp no)
+		(fields_autoplaced yes)
 		(property "Reference" "D26"
-			(at 237.49 135.89 0)
+			(at 237.49 142.24 0)
 			(show_name no)
 			(do_not_autoplace no)
@@
 			)
 		)
-		(property "Value" "RB521S30T1G"
+		(property "Value" "PMEG3010CEJ,115"
 			(at 217.17 123.19 0)
 			(hide yes)
@@
 			)
 		)
-		(property "Footprint" "antmicro-footprints:SOD-523"
+		(property "Footprint" "antmicro-footprints:D_SOD-323F"
 			(at 217.17 128.27 0)
 			(hide yes)
@@
 			)
 		)
-		(property "Datasheet" "https://www.onsemi.com/pdf/datasheet/rb521s30t1-d.pdf"
+		(property "Datasheet" "https://assets.nexperia.com/documents/data-sheet/PMEG3010CEH_PMEG3010CEJ.pdf"
 			(at 217.17 125.73 0)
 			(hide yes)
@@
 			)
 		)
-		(property "Description" "Small Signal Schottky Diode, Single, 30 V, 200 mA, 500 mV, 1 A, 125 °C"
+		(property "Description" "Schottky Rectifier, 30 V, 1 A, Single, SOD-323F, 2 Pins, 520 mV"
 			(at 240.03 138.43 0)
 			(hide yes)
@@
 					(size 1.27 1.27)
 				)
+				(justify left bottom)
 			)
 		)
-		(property "MPN" "RB521S30T1G"
-			(at 237.49 140.97 0)
+		(property "MPN" "PMEG3010CEJ,115"
+			(at 237.49 144.78 0)
 			(show_name no)
 			(do_not_autoplace no)
@@
 			)
 		)
-		(property "Manufacturer" "ON Semiconductor"
+		(property "Manufacturer" "Nexperia"
 			(at 217.17 120.65 0)
 			(hide yes)

Commit message: [#101340] Change C240 to 4.7uF
Re-use 4.7uF from other sheets
Parts:
- C240: value C_2u2_0402 -> C_4u7_0402; symbol antmicroCapacitors0402:C_2u2_0402 -> antmicroCapacitors0402:C_4u7_0402; MPN C1005X5R1A225K050BC -> GRM155R61A475MEAAD; Manufacturer TDK -> Murata; Val 2u2 -> 4u7
Changed lines of the file:
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@@
 	)
 	(symbol
-		(lib_id "antmicroCapacitors0402:C_2u2_0402")
+		(lib_id "antmicroCapacitors0402:C_4u7_0402")
 		(at 128.27 106.68 90)
 		(unit 1)
@@
 			)
 		)
-		(property "Value" "C_2u2_0402"
+		(property "Value" "C_4u7_0402"
 			(at 138.43 86.36 0)
 			(hide yes)
@@
 			)
 		)
-		(property "Datasheet" "https://product.tdk.com/en/search/capacitor/ceramic/mlcc/info?part_no=C1005X5R1A225K050BC"
+		(property "Datasheet" "https://www.murata.com/products/productdetail?partno=GRM155R61A475MEAA%23"
 			(at 143.51 86.36 0)
 			(hide yes)
@@
 			)
 		)
-		(property "Description" "SMD Multilayer Ceramic Capacitor, 2.2 µF, 10 V, 0402 [1005 Metric], ± 10%, X5R, C"
+		(property "Description" "SMD Multilayer Ceramic Capacitor, 4.7 µF, 10 V, 0402 [1005 Metric], ± 20%, X5R, GRM Series"
 			(at 161.29 86.36 0)
 			(hide yes)
@@
 			)
 		)
-		(property "MPN" "C1005X5R1A225K050BC"
+		(property "MPN" "GRM155R61A475MEAAD"
 			(at 146.05 86.36 0)
 			(hide yes)
@@
 			)
 		)
-		(property "Manufacturer" "TDK"
+		(property "Manufacturer" "Murata"
 			(at 148.59 86.36 0)
 			(hide yes)
@@
 			)
 		)
-		(property "Val" "2u2"
+		(property "Val" "4u7"
 			(at 129.032 106.172 90)
 			(show_name no)

Commit message: [#101340] Reduce number of unique R MPNs
Parts:
- R347: value R_1M_0402 -> R_887k_0402; symbol antmicroResistors0402:R_1M_0402 -> antmicroResistors0402:R_887k_0402; MPN CR0402-FX-1004GLF -> ERJ-2RKF8873X; Manufacturer Bourns -> Panasonic; Val 1M -> 887k
Changed lines of the file:
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@@
 	)
 	(symbol
-		(lib_id "antmicroResistors0402:R_1M_0402")
+		(lib_id "antmicroResistors0402:R_887k_0402")
 		(at 306.07 151.13 90)
 		(unit 1)
@@
 			)
 		)
-		(property "Value" "R_1M_0402"
+		(property "Value" "R_887k_0402"
 			(at 318.77 130.81 0)
 			(hide yes)
@@
 			)
 		)
-		(property "Datasheet" "https://www.bourns.com/docs/product-datasheets/cr.pdf"
+		(property "Datasheet" "https://eu.mouser.com/datasheet/2/315/AOA0000C304-1149620.pdf"
 			(at 323.85 130.81 0)
 			(hide yes)
@@
 			)
 		)
-		(property "Description" "SMD Chip Resistor, 1 Mohm, ± 1%, 62.5 mW, 0402 [1005 Metric], Thick Film, General Purpose"
+		(property "Description" "SMD Chip Resistor"
 			(at 306.07 151.13 0)
 			(hide yes)
@@
 			)
 		)
-		(property "MPN" "CR0402-FX-1004GLF"
+		(property "MPN" "ERJ-2RKF8873X"
 			(at 326.39 130.81 0)
 			(hide yes)
@@
 			)
 		)
-		(property "Manufacturer" "Bourns"
+		(property "Manufacturer" "Panasonic"
 			(at 328.93 130.81 0)
 			(hide yes)
@@
 			)
 		)
-		(property "Val" "1M"
+		(property "Val" "887k"
 			(at 307.34 149.86 90)
 			(show_name no)
