File: bios.kicad_sch (KiCad schematic)
At the start: 39 parts, among them U12 TMUX1574RSVR, U13 MT25QU01GBBB8_SOIC, U14 TMUX1574RSVR, U15 MT25QU01GBBB8_SOIC

Commit message: [#101340] Add flash sockets
Parts:
- added J1201, J1202: Socket_SOP2-16_ACA-SPI-006-K01_Flash_CUSTOM, antmicro-footprints:Socket_SOP2-16_ACA-SPI-006-K01, symbol antmicroMechanicalParts:Socket_SOP2-16_ACA-SPI-006-K01_Flash_CUSTOM
- U13, U15: now not fitted
Connections:
- net +1V8: now also J1201.2 (VCC), J1202.2 (VCC)
- net GND: now also J1201.10 (VSS), J1202.10 (VSS)
- net at R161.2, U15.15 (SI/IO0): now also J1202.15 (SI/IO0)
- net at R158.2, U15.3 (~{RESET}): now also J1202.3 (~{RESET})
- net at R160.2, U15.7 (~{CS}): now also J1202.7 (~{CS})
- net at R164.2, U15.1 (~{HOLD/IO3}): now also J1202.1 (~{HOLD/IO3})
- net at U15.14 (VIO): now also J1202.14 (VIO)
- net at R159.2, U15.16 (SCK): now also J1202.16 (SCK)
- net at R162.2, U15.8 (SO/IO1): now also J1202.8 (SO/IO1)
- net at R163.2, U15.9 (~{WP/IO2}): now also J1202.9 (~{WP/IO2})
- net at R155.2, U13.1 (~{HOLD/IO3}): now also J1201.1 (~{HOLD/IO3})
- net at U13.14 (VIO): now also J1201.14 (VIO)
- net at R152.2, U13.15 (SI/IO0): now also J1201.15 (SI/IO0)
- net at R150.2, U13.16 (SCK): now also J1201.16 (SCK)
- net at R149.2, U13.3 (~{RESET}): now also J1201.3 (~{RESET})
- net at R151.2, U13.7 (~{CS}): now also J1201.7 (~{CS})
- net at R153.2, U13.8 (SO/IO1): now also J1201.8 (SO/IO1)
- net at R154.2, U13.9 (~{WP/IO2}): now also J1201.9 (~{WP/IO2})
- no-connect marks 10 -> 8
Other:
- moved on the sheet: C91, C93, R148, R149, R150, R151, R152, R153, R154, R155, R157, R158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

Commit message: [#101340] Unify BIOS resistors
Change 4.7Ohm to 33Ohm
Parts:
- R152, R153, R154, R155, R161, R162, R163, R164: value R_4R7_0402 -> R_33R_0402; symbol antmicroResistors0402:R_4R7_0402 -> antmicroResistors0402:R_33R_0402; MPN CR0402-FX-4R70GLF -> CR0402-FX-33R0GLF; Val 4R7 -> 33R
Changed lines of the file:
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@@
 	)
 	(symbol
-		(lib_id "antmicroResistors0402:R_4R7_0402")
+		(lib_id "antmicroResistors0402:R_33R_0402")
 		(at 208.28 121.92 0)
 		(unit 1)
@@
 			)
 		)
-		(property "Value" "R_4R7_0402"
+		(property "Value" "R_33R_0402"
 			(at 228.6 134.62 0)
 			(hide yes)
@@
 			)
 		)
-		(property "Description" "SMD Chip Resistor, 4.7 ohm, ± 1%, 62.5 mW, 0402 [1005 Metric], Thick Film, General Purpose"
+		(property "Description" "SMD Chip Resistor, 33 ohm, ± 1%, 62.5 mW, 0402 [1005 Metric], Thick Film, General Purpose"
 			(at 228.6 152.4 0)
 			(hide yes)
@@
 			)
 		)
-		(property "MPN" "CR0402-FX-4R70GLF"
+		(property "MPN" "CR0402-FX-33R0GLF"
 			(at 228.6 142.24 0)
 			(hide yes)
@@
 			)
 		)
-		(property "Val" "4R7"
+		(property "Val" "33R"
 			(at 213.36 120.65 0)
 			(show_name no)
@@
 	)
 	(symbol
-		(lib_id "antmicroResistors0402:R_4R7_0402")
+		(lib_id "antmicroResistors0402:R_33R_0402")
 		(at 208.28 66.04 0)
 		(unit 1)
@@
 			)
 		)
-		(property "Value" "R_4R7_0402"
+		(property "Value" "R_33R_0402"
 			(at 228.6 78.74 0)
 			(hide yes)
@@
 			)
 		)
-		(property "Description" "SMD Chip Resistor, 4.7 ohm, ± 1%, 62.5 mW, 0402 [1005 Metric], Thick Film, General Purpose"
+		(property "Description" "SMD Chip Resistor, 33 ohm, ± 1%, 62.5 mW, 0402 [1005 Metric], Thick Film, General Purpose"
 			(at 228.6 96.52 0)
 			(hide yes)
@@
 			)
 		)
-		(property "MPN" "CR0402-FX-4R70GLF"
+		(property "MPN" "CR0402-FX-33R0GLF"
 			(at 228.6 86.36 0)
 			(hide yes)
@@
 			)
 		)
-		(property "Val" "4R7"
+		(property "Val" "33R"
 			(at 213.36 64.77 0)
 			(show_name no)
@@
 	)
 	(symbol
-		(lib_id "antmicroResistors0402:R_4R7_0402")
+		(lib_id "antmicroResistors0402:R_33R_0402")
 		(at 208.28 129.54 0)
 		(unit 1)
@@
 			)
 		)
-		(property "Value" "R_4R7_0402"
+		(property "Value" "R_33R_0402"
 			(at 228.6 142.24 0)
 			(hide yes)
@@
 			)
 		)
-		(property "Description" "SMD Chip Resistor, 4.7 ohm, ± 1%, 62.5 mW, 0402 [1005 Metric], Thick Film, General Purpose"
+		(property "Description" "SMD Chip Resistor, 33 ohm, ± 1%, 62.5 mW, 0402 [1005 Metric], Thick Film, General Purpose"
 			(at 228.6 160.02 0)
 			(hide yes)
@@
 			)
 		)
-		(property "MPN" "CR0402-FX-4R70GLF"
+		(property "MPN" "CR0402-FX-33R0GLF"
 			(at 228.6 149.86 0)
 			(hide yes)
@@
 			)
 		)
-		(property "Val" "4R7"
+		(property "Val" "33R"
 			(at 213.36 128.27 0)
 			(show_name no)
@@
 	)
 	(symbol
-		(lib_id "antmicroResistors0402:R_4R7_0402")
+		(lib_id "antmicroResistors0402:R_33R_0402")
 		(at 208.28 124.46 0)
 		(unit 1)
@@
 			)
 		)
-		(property "Value" "R_4R7_0402"
+		(property "Value" "R_33R_0402"
 			(at 228.6 137.16 0)
 			(hide yes)
@@
 			)
 		)
-		(property "Description" "SMD Chip Resistor, 4.7 ohm, ± 1%, 62.5 mW, 0402 [1005 Metric], Thick Film, General Purpose"
+		(property "Description" "SMD Chip Resistor, 33 ohm, ± 1%, 62.5 mW, 0402 [1005 Metric], Thick Film, General Purpose"
 			(at 228.6 154.94 0)
 			(hide yes)
@@
 			)
 		)
-		(property "MPN" "CR0402-FX-4R70GLF"
+		(property "MPN" "CR0402-FX-33R0GLF"
 			(at 228.6 144.78 0)
 			(hide yes)
@@
 			)
 		)
-		(property "Val" "4R7"
+		(property "Val" "33R"
 			(at 213.36 123.19 0)
 			(show_name no)
@@
 	)
 	(symbol
-		(lib_id "antmicroResistors0402:R_4R7_0402")
+		(lib_id "antmicroResistors0402:R_33R_0402")
 		(at 208.28 63.5 0)
 		(unit 1)
@@
 			)
 		)
-		(property "Value" "R_4R7_0402"
+		(property "Value" "R_33R_0402"
 			(at 228.6 76.2 0)
 			(hide yes)
@@
 			)
 		)
-		(property "Description" "SMD Chip Resistor, 4.7 ohm, ± 1%, 62.5 mW, 0402 [1005 Metric], Thick Film, General Purpose"
+		(property "Description" "SMD Chip Resistor, 33 ohm, ± 1%, 62.5 mW, 0402 [1005 Metric], Thick Film, General Purpose"
 			(at 228.6 93.98 0)
 			(hide yes)
@@
 			)
 		)
-		(property "MPN" "CR0402-FX-4R70GLF"
+		(property "MPN" "CR0402-FX-33R0GLF"
 			(at 228.6 83.82 0)
 			(hide yes)
@@
 			)
 		)
-		(property "Val" "4R7"
+		(property "Val" "33R"
 			(at 213.36 62.23 0)
 			(show_name no)
@@
 	)
 	(symbol
-		(lib_id "antmicroResistors0402:R_4R7_0402")
+		(lib_id "antmicroResistors0402:R_33R_0402")
 		(at 208.28 127 0)
 		(unit 1)
@@
 			)
 		)
-		(property "Value" "R_4R7_0402"
+		(property "Value" "R_33R_0402"
 			(at 228.6 139.7 0)
 			(hide yes)
@@
 			)
 		)
-		(property "Description" "SMD Chip Resistor, 4.7 ohm, ± 1%, 62.5 mW, 0402 [1005 Metric], Thick Film, General Purpose"
+		(property "Description" "SMD Chip Resistor, 33 ohm, ± 1%, 62.5 mW, 0402 [1005 Metric], Thick Film, General Purpose"
 			(at 228.6 157.48 0)
 			(hide yes)
@@
 			)
 		)
-		(property "MPN" "CR0402-FX-4R70GLF"
+		(property "MPN" "CR0402-FX-33R0GLF"
 			(at 228.6 147.32 0)
 			(hide yes)
@@
 			)
 		)
-		(property "Val" "4R7"
+		(property "Val" "33R"
 			(at 213.36 125.73 0)
 			(show_name no)
@@
 	)
 	(symbol
-		(lib_id "antmicroResistors0402:R_4R7_0402")
+		(lib_id "antmicroResistors0402:R_33R_0402")
 		(at 208.28 58.42 0)
 		(unit 1)
@@
 			)
 		)
-		(property "Value" "R_4R7_0402"
+		(property "Value" "R_33R_0402"
 			(at 228.6 71.12 0)
 			(hide yes)
@@
 			)
 		)
-		(property "Description" "SMD Chip Resistor, 4.7 ohm, ± 1%, 62.5 mW, 0402 [1005 Metric], Thick Film, General Purpose"
+		(property "Description" "SMD Chip Resistor, 33 ohm, ± 1%, 62.5 mW, 0402 [1005 Metric], Thick Film, General Purpose"
 			(at 228.6 88.9 0)
 			(hide yes)
@@
 			)
 		)
-		(property "MPN" "CR0402-FX-4R70GLF"
+		(property "MPN" "CR0402-FX-33R0GLF"
 			(at 228.6 78.74 0)
 			(hide yes)
@@
 			)
 		)
-		(property "Val" "4R7"
+		(property "Val" "33R"
 			(at 213.36 57.15 0)
 			(show_name no)
@@
 	)
 	(symbol
-		(lib_id "antmicroResistors0402:R_4R7_0402")
+		(lib_id "antmicroResistors0402:R_33R_0402")
 		(at 208.28 60.96 0)
 		(unit 1)
@@
 			)
 		)
-		(property "Value" "R_4R7_0402"
+		(property "Value" "R_33R_0402"
 			(at 228.6 73.66 0)
 			(hide yes)
@@
 			)
 		)
-		(property "Description" "SMD Chip Resistor, 4.7 ohm, ± 1%, 62.5 mW, 0402 [1005 Metric], Thick Film, General Purpose"
+		(property "Description" "SMD Chip Resistor, 33 ohm, ± 1%, 62.5 mW, 0402 [1005 Metric], Thick Film, General Purpose"
 			(at 228.6 91.44 0)
 			(hide yes)
@@
 			)
 		)
-		(property "MPN" "CR0402-FX-4R70GLF"
+		(property "MPN" "CR0402-FX-33R0GLF"
 			(at 228.6 81.28 0)
 			(hide yes)
@@
 			)
 		)
-		(property "Val" "4R7"
+		(property "Val" "33R"
 			(at 213.36 59.69 0)
 			(show_name no)

Commit message: [#101340] Add comments to ERC/DRC exclusions
Connections:
- net BIOS1_NC: now reaches U15.13 (NC)
- net BIOS1_NC: now also J1202.13 (NC)
- net BIOS1_VIO: now reaches J1202.14 (VIO), U15.14 (VIO)
- net BIOS1_RFU: now reaches U15.6 (RFU)
- net BIOS1_RFU: now also J1202.6 (RFU)
- net BIOS0_NC: now reaches U13.13 (NC)
- net BIOS0_NC: now also J1201.13 (NC)
- net BIOS0_VIO: now reaches J1201.14 (VIO), U13.14 (VIO)
- net BIOS0_RFU: now reaches U13.6 (RFU)
- net BIOS0_RFU: now also J1201.6 (RFU)
- net BIOS0_DNU2: now reaches J1201.11 (DNU)
- net BIOS0_DNU2: now also U13.11 (DNU)
- net BIOS0_DNU3: now reaches J1201.12 (DNU)
- net BIOS0_DNU3: now also U13.12 (DNU)
- net BIOS0_DNU0: now reaches J1201.4 (DNU)
- net BIOS0_DNU0: now also U13.4 (DNU)
- net BIOS0_DNU1: now reaches J1201.5 (DNU)
- net BIOS0_DNU1: now also U13.5 (DNU)
- net BIOS1_DNU2: now reaches J1202.11 (DNU)
- net BIOS1_DNU2: now also U15.11 (DNU)
- net BIOS1_DNU3: now reaches J1202.12 (DNU)
- net BIOS1_DNU3: now also U15.12 (DNU)
- net BIOS1_DNU0: now reaches J1202.4 (DNU)
- net BIOS1_DNU0: now also U15.4 (DNU)
- net BIOS1_DNU1: now reaches J1202.5 (DNU)
- net BIOS1_DNU1: now also U15.5 (DNU)
